File: uHoubolt_PCB_PMU/balancer.sch (KiCad schematic (older format))
At the start: 25 parts, among them Q3 BUK7M27-80EX, Q4 BUK7M27-80EX, U9 BQ77915

Commit message: add current measurement
Parts:
- added C? (x3): 0.1uF, symbol Device:C_Small
- added R? (x2): 100, symbol Device:R_Small
- R29, R30, R31, R32: value 33 -> 134
- R33: value R_Small -> 3m
- R34: value R_Small -> 4.5k
- R40: value 1M -> 3.3M
Connections:
- net labels added: VSS
- wire segments 92 -> 96
Other:
- moved on the sheet: R29, R33

Commit message: add resistor values of regulator
Connections:
- wire segments 96 -> 97
Other:
- moved on the sheet: D?
Changed lines of the file:
@@
 AR Path="/601B6EED" Ref="R?"  Part="1"
 AR Path="/6017800E/601B6EED" Ref="R39"  Part="1"
-F 0 "R39" V 6150 3600 50  0000 C CNN
-F 1 "1M" V 6050 3600 50  0000 C CNN
+F 0 "R39" V 6225 3600 50  0000 C CNN
+F 1 "1M" V 6150 3575 50  0000 C CNN
 F 2 "" H 6100 3700 50  0001 C CNN
 F 3 "~" H 6100 3700 50  0001 C CNN
@@
 L power:GND #PWR?
 U 1 1 601B6F84
-P 6050 3300
+P 6125 3300
 AR Path="/601B6F84" Ref="#PWR?"  Part="1"
 AR Path="/6017800E/601B6F84" Ref="#PWR0173"  Part="1"
-F 0 "#PWR0173" H 6050 3050 50  0001 C CNN
-F 1 "GND" V 6055 3172 50  0000 R CNN
-F 2 "" H 6050 3300 50  0001 C CNN
-F 3 "" H 6050 3300 50  0001 C CNN
-	1    6050 3300
+F 0 "#PWR0173" H 6125 3050 50  0001 C CNN
+F 1 "GND" V 6130 3172 50  0000 R CNN
+F 2 "" H 6125 3300 50  0001 C CNN
+F 3 "" H 6125 3300 50  0001 C CNN
+	1    6125 3300
 	0    -1   -1   0
 $EndComp
@@
 AR Path="/601B6F8A" Ref="R?"  Part="1"
 AR Path="/6017800E/601B6F8A" Ref="R38"  Part="1"
-F 0 "R38" V 5900 3300 50  0000 C CNN
-F 1 "100k" V 6000 3350 50  0000 C CNN
+F 0 "R38" V 5900 3450 50  0000 C CNN
+F 1 "100k" V 6000 3425 50  0000 C CNN
 F 2 "" H 5950 3300 50  0001 C CNN
 F 3 "~" H 5950 3300 50  0001 C CNN
@@
 AR Path="/601B6F90" Ref="R?"  Part="1"
 AR Path="/6017800E/601B6F90" Ref="R37"  Part="1"
-F 0 "R37" V 5900 3150 50  0000 C CNN
+F 0 "R37" V 5900 3250 50  0000 C CNN
 F 1 "10k" V 6000 3200 50  0000 C CNN
 F 2 "" H 5950 3100 50  0001 C CNN
@@
 L Device:D_Zener D?
 U 1 1 5FF7203B
-P 6050 4050
-F 0 "D?" H 6050 3834 50  0000 C CNN
-F 1 "D_Zener" H 6050 3925 50  0000 C CNN
-F 2 "" H 6050 4050 50  0001 C CNN
-F 3 "~" H 6050 4050 50  0001 C CNN
-	1    6050 4050
+P 6050 4125
+F 0 "D?" H 6050 3909 50  0000 C CNN
+F 1 "D_Zener" H 6050 4000 50  0000 C CNN
+F 2 "" H 6050 4125 50  0001 C CNN
+F 3 "~" H 6050 4125 50  0001 C CNN
+	1    6050 4125
 	-1   0    0    1
 $EndComp
-Wire Wire Line
-	6250 3700 6250 4050
-Wire Wire Line
-	6250 4050 6200 4050
 Connection ~ 6250 3700
 Wire Wire Line
 	6250 3700 6300 3700
-Wire Wire Line
-	5850 3700 5850 4050
-Wire Wire Line
-	5850 4050 5900 4050
 Connection ~ 5850 3700
 Wire Wire Line
@@
 AR Path="/60039E54" Ref="C?"  Part="1"
 AR Path="/6017800E/60039E54" Ref="C?"  Part="1"
-F 0 "C?" H 4792 4196 50  0000 L CNN
-F 1 "0.1uF" H 4792 4105 50  0000 L CNN
+F 0 "C?" H 4800 4150 50  0000 L CNN
+F 1 "0.1uF" H 4775 4075 50  0000 L CNN
 F 2 "" H 4700 4150 50  0001 C CNN
 F 3 "~" H 4700 4150 50  0001 C CNN
@@
 AR Path="/600493FC" Ref="C?"  Part="1"
 AR Path="/6017800E/600493FC" Ref="C?"  Part="1"
-F 0 "C?" H 4392 4096 50  0000 L CNN
-F 1 "0.1uF" H 4392 4005 50  0000 L CNN
+F 0 "C?" V 4525 3975 50  0000 L CNN
+F 1 "0.1uF" V 4450 3850 50  0000 L CNN
 F 2 "" H 4300 4050 50  0001 C CNN
 F 3 "~" H 4300 4050 50  0001 C CNN
@@
 Wire Wire Line
 	5850 3400 6500 3400
+Wire Wire Line
+	6200 4125 6250 4125
+Wire Wire Line
+	6250 3700 6250 4125
+Wire Wire Line
+	5850 4125 5900 4125
+Wire Wire Line
+	5850 3700 5850 4125
+Wire Wire Line
+	6050 3300 6125 3300
 $EndSCHEMATC

Commit message: connect labels to muC
Parts:
- gave numbers to parts that had none: 7
- renumbered C38 to C39, C39 to C40, C40 to C42, R28 to R30, R30 to R31, R31 to R32, R32 to R33, R33 to R35, R34 to R37, R35 to R38, R36 to R39, R37 to R40, R38 to R41, R39 to R42, R40 to R43, R41 to R44
Connections:
- net labels added: CBI
- net labels removed: VSS
Changed lines of the file:
@@
 P 4800 2700
 AR Path="/601B6EC5" Ref="C?"  Part="1"
-AR Path="/6017800E/601B6EC5" Ref="C40"  Part="1"
-F 0 "C40" V 4850 2500 50  0000 L CNN
+AR Path="/6017800E/601B6EC5" Ref="C42"  Part="1"
+F 0 "C42" V 4850 2500 50  0000 L CNN
 F 1 "1uF" V 4950 2500 50  0000 L CNN
 F 2 "" H 4800 2700 50  0001 C CNN
@@
 P 4200 2500
 AR Path="/601B6ECB" Ref="#PWR?"  Part="1"
-AR Path="/6017800E/601B6ECB" Ref="#PWR0169"  Part="1"
-F 0 "#PWR0169" H 4200 2250 50  0001 C CNN
+AR Path="/6017800E/601B6ECB" Ref="#PWR066"  Part="1"
+F 0 "#PWR066" H 4200 2250 50  0001 C CNN
 F 1 "GND" H 4150 2400 50  0000 R CNN
 F 2 "" H 4200 2500 50  0001 C CNN
@@
 P 6450 3800
 AR Path="/601B6EE7" Ref="R?"  Part="1"
-AR Path="/6017800E/601B6EE7" Ref="R40"  Part="1"
-F 0 "R40" H 6400 3900 50  0000 R CNN
+AR Path="/6017800E/601B6EE7" Ref="R43"  Part="1"
+F 0 "R43" H 6400 3900 50  0000 R CNN
 F 1 "3.3M" H 6400 4000 50  0000 R CNN
 F 2 "" H 6450 3800 50  0001 C CNN
@@
 P 6100 3700
 AR Path="/601B6EED" Ref="R?"  Part="1"
-AR Path="/6017800E/601B6EED" Ref="R39"  Part="1"
-F 0 "R39" V 6225 3600 50  0000 C CNN
+AR Path="/6017800E/601B6EED" Ref="R42"  Part="1"
+F 0 "R42" V 6225 3600 50  0000 C CNN
 F 1 "1M" V 6150 3575 50  0000 C CNN
 F 2 "" H 6100 3700 50  0001 C CNN
@@
 P 6700 3600
 AR Path="/601B6EF6" Ref="R?"  Part="1"
-AR Path="/6017800E/601B6EF6" Ref="R41"  Part="1"
-F 0 "R41" V 6800 3600 50  0000 C CNN
+AR Path="/6017800E/601B6EF6" Ref="R44"  Part="1"
+F 0 "R44" V 6800 3600 50  0000 C CNN
 F 1 "470k" V 6900 3650 50  0000 C CNN
 F 2 "" H 6700 3600 50  0001 C CNN
@@
 P 5500 4000
 AR Path="/601B6EFF" Ref="R?"  Part="1"
-AR Path="/6017800E/601B6EFF" Ref="R35"  Part="1"
-F 0 "R35" H 5400 3950 50  0000 R CNN
+AR Path="/6017800E/601B6EFF" Ref="R38"  Part="1"
+F 0 "R38" H 5400 3950 50  0000 R CNN
 F 1 "1M" H 5441 4045 50  0000 R CNN
 F 2 "" H 5500 4000 50  0001 C CNN
@@
 P 5350 3900
 AR Path="/601B6F07" Ref="R?"  Part="1"
-AR Path="/6017800E/601B6F07" Ref="R34"  Part="1"
-F 0 "R34" V 5450 3850 50  0000 C CNN
+AR Path="/6017800E/601B6F07" Ref="R37"  Part="1"
+F 0 "R37" V 5450 3850 50  0000 C CNN
 F 1 "4.5k" V 5550 3800 50  0000 C CNN
 F 2 "" H 5350 3900 50  0001 C CNN
@@
 P 4400 4500
 AR Path="/601B6F1C" Ref="R?"  Part="1"
-AR Path="/6017800E/601B6F1C" Ref="R33"  Part="1"
-F 0 "R33" V 4500 4500 50  0000 C CNN
+AR Path="/6017800E/601B6F1C" Ref="R35"  Part="1"
+F 0 "R35" V 4500 4500 50  0000 C CNN
 F 1 "3m" V 4600 4500 50  0000 C CNN
 F 2 "" H 4400 4500 50  0001 C CNN
@@
 P 3100 4850
 AR Path="/601B6F24" Ref="#PWR?"  Part="1"
-AR Path="/6017800E/601B6F24" Ref="#PWR0170"  Part="1"
-F 0 "#PWR0170" H 3100 4600 50  0001 C CNN
+AR Path="/6017800E/601B6F24" Ref="#PWR064"  Part="1"
+F 0 "#PWR064" H 3100 4600 50  0001 C CNN
 F 1 "GND" H 3105 4677 50  0000 C CNN
 F 2 "" H 3100 4850 50  0001 C CNN
@@
 P 4400 3500
 AR Path="/601B6F33" Ref="#PWR?"  Part="1"
-AR Path="/6017800E/601B6F33" Ref="#PWR0171"  Part="1"
-F 0 "#PWR0171" H 4400 3250 50  0001 C CNN
+AR Path="/6017800E/601B6F33" Ref="#PWR067"  Part="1"
+F 0 "#PWR067" H 4400 3250 50  0001 C CNN
 F 1 "GND" V 4405 3372 50  0000 R CNN
 F 2 "" H 4400 3500 50  0001 C CNN
@@
 P 4400 3600
 AR Path="/601B6F39" Ref="C?"  Part="1"
-AR Path="/6017800E/601B6F39" Ref="C39"  Part="1"
-F 0 "C39" H 4492 3646 50  0000 L CNN
+AR Path="/6017800E/601B6F39" Ref="C40"  Part="1"
+F 0 "C40" H 4492 3646 50  0000 L CNN
 F 1 "1uF" H 4492 3555 50  0000 L CNN
 F 2 "" H 4400 3600 50  0001 C CNN
@@
 P 4400 3400
 AR Path="/601B6F41" Ref="C?"  Part="1"
-AR Path="/6017800E/601B6F41" Ref="C38"  Part="1"
-F 0 "C38" H 4492 3446 50  0000 L CNN
+AR Path="/6017800E/601B6F41" Ref="C39"  Part="1"
+F 0 "C39" H 4492 3446 50  0000 L CNN
 F 1 "1uF" H 4492 3355 50  0000 L CNN
 F 2 "" H 4400 3400 50  0001 C CNN
@@
 P 5950 2800
 AR Path="/601B6F67" Ref="R?"  Part="1"
-AR Path="/6017800E/601B6F67" Ref="R36"  Part="1"
-F 0 "R36" V 6000 2650 50  0000 C CNN
+AR Path="/6017800E/601B6F67" Ref="R39"  Part="1"
+F 0 "R39" V 6000 2650 50  0000 C CNN
 F 1 "10k" V 5900 2650 50  0000 C CNN
 F 2 "" H 5950 2800 50  0001 C CNN
@@
 P 7150 3200
 AR Path="/601B6F6E" Ref="#PWR?"  Part="1"
-AR Path="/6017800E/601B6F6E" Ref="#PWR0172"  Part="1"
-F 0 "#PWR0172" H 7150 2950 50  0001 C CNN
+AR Path="/6017800E/601B6F6E" Ref="#PWR071"  Part="1"
+F 0 "#PWR071" H 7150 2950 50  0001 C CNN
 F 1 "GND" V 7155 3072 50  0000 R CNN
 F 2 "" H 7150 3200 50  0001 C CNN
@@
 P 6125 3300
 AR Path="/601B6F84" Ref="#PWR?"  Part="1"
-AR Path="/6017800E/601B6F84" Ref="#PWR0173"  Part="1"
-F 0 "#PWR0173" H 6125 3050 50  0001 C CNN
+AR Path="/6017800E/601B6F84" Ref="#PWR069"  Part="1"
+F 0 "#PWR069" H 6125 3050 50  0001 C CNN
 F 1 "GND" V 6130 3172 50  0000 R CNN
 F 2 "" H 6125 3300 50  0001 C CNN
@@
 P 5950 3300
 AR Path="/601B6F8A" Ref="R?"  Part="1"
-AR Path="/6017800E/601B6F8A" Ref="R38"  Part="1"
-F 0 "R38" V 5900 3450 50  0000 C CNN
+AR Path="/6017800E/601B6F8A" Ref="R41"  Part="1"
+F 0 "R41" V 5900 3450 50  0000 C CNN
 F 1 "100k" V 6000 3425 50  0000 C CNN
 F 2 "" H 5950 3300 50  0001 C CNN
@@
 P 5950 3100
 AR Path="/601B6F90" Ref="R?"  Part="1"
-AR Path="/6017800E/601B6F90" Ref="R37"  Part="1"
-F 0 "R37" V 5900 3250 50  0000 C CNN
+AR Path="/6017800E/601B6F90" Ref="R40"  Part="1"
+F 0 "R40" V 5900 3250 50  0000 C CNN
 F 1 "10k" V 6000 3200 50  0000 C CNN
 F 2 "" H 5950 3100 50  0001 C CNN
@@
 P 4050 3750
 AR Path="/601B6F96" Ref="R?"  Part="1"
-AR Path="/6017800E/601B6F96" Ref="R31"  Part="1"
-F 0 "R31" V 3854 3750 50  0000 C CNN
+AR Path="/6017800E/601B6F96" Ref="R32"  Part="1"
+F 0 "R32" V 3854 3750 50  0000 C CNN
 F 1 "134" V 3945 3750 50  0000 C CNN
 F 2 "" H 4050 3750 50  0001 C CNN
@@
 P 4050 3300
 AR Path="/601B6F9C" Ref="R?"  Part="1"
-AR Path="/6017800E/601B6F9C" Ref="R30"  Part="1"
-F 0 "R30" V 4100 3150 50  0000 C CNN
+AR Path="/6017800E/601B6F9C" Ref="R31"  Part="1"
+F 0 "R31" V 4100 3150 50  0000 C CNN
 F 1 "134" V 4200 3150 50  0000 C CNN
 F 2 "" H 4050 3300 50  0001 C CNN
@@
 P 4200 2900
 AR Path="/601B6FAF" Ref="R?"  Part="1"
-AR Path="/6017800E/601B6FAF" Ref="R32"  Part="1"
-F 0 "R32" V 4000 2850 50  0000 C CNN
+AR Path="/6017800E/601B6FAF" Ref="R33"  Part="1"
+F 0 "R33" V 4000 2850 50  0000 C CNN
 F 1 "134" V 4100 2850 50  0000 C CNN
 F 2 "" H 4200 2900 50  0001 C CNN
@@
 P 6150 2700
 AR Path="/601B6FBD" Ref="#PWR?"  Part="1"
-AR Path="/6017800E/601B6FBD" Ref="#PWR0174"  Part="1"
-F 0 "#PWR0174" H 6150 2450 50  0001 C CNN
+AR Path="/6017800E/601B6FBD" Ref="#PWR070"  Part="1"
+F 0 "#PWR070" H 6150 2450 50  0001 C CNN
 F 1 "GND" V 6155 2572 50  0000 R CNN
 F 2 "" H 6150 2700 50  0001 C CNN
@@
 P 3950 2300
 AR Path="/601B6FC9" Ref="R?"  Part="1"
-AR Path="/6017800E/601B6FC9" Ref="R28"  Part="1"
-F 0 "R28" V 3754 2300 50  0000 C CNN
+AR Path="/6017800E/601B6FC9" Ref="R30"  Part="1"
+F 0 "R30" V 3754 2300 50  0000 C CNN
 F 1 "1k" V 3845 2300 50  0000 C CNN
 F 2 "" H 3950 2300 50  0001 C CNN
@@
 NoConn ~ 5850 2900
 $Comp
-L Device:Thermistor_NTC TH?
+L Device:Thermistor_NTC TH1
 U 1 1 5FF5E99E
 P 6500 3200
-F 0 "TH?" V 6210 3200 50  0000 C CNN
+F 0 "TH1" V 6210 3200 50  0000 C CNN
 F 1 "Thermistor_NTC" V 6301 3200 50  0000 C CNN
 F 2 "" H 6500 3250 50  0001 C CNN
@@
 	6650 3200 7050 3200
 $Comp
-L Device:D_Zener D?
+L Device:D_Zener D6
 U 1 1 5FF7203B
 P 6050 4125
-F 0 "D?" H 6050 3909 50  0000 C CNN
+F 0 "D6" H 6050 3909 50  0000 C CNN
 F 1 "D_Zener" H 6050 4000 50  0000 C CNN
 F 2 "" H 6050 4125 50  0001 C CNN
@@
 P 3700 4150
 AR Path="/600073DA" Ref="C?"  Part="1"
-AR Path="/6017800E/600073DA" Ref="C?"  Part="1"
-F 0 "C?" H 3792 4196 50  0000 L CNN
+AR Path="/6017800E/600073DA" Ref="C34"  Part="1"
+F 0 "C34" H 3792 4196 50  0000 L CNN
 F 1 "0.1uF" H 3792 4105 50  0000 L CNN
 F 2 "" H 3700 4150 50  0001 C CNN
@@
 P 4200 4150
 AR Path="/60007E4C" Ref="R?"  Part="1"
-AR Path="/6017800E/60007E4C" Ref="R?"  Part="1"
-F 0 "R?" V 4250 4000 50  0000 C CNN
+AR Path="/6017800E/60007E4C" Ref="R34"  Part="1"
+F 0 "R34" V 4250 4000 50  0000 C CNN
 F 1 "100" V 4150 4000 50  0000 C CNN
 F 2 "" H 4200 4150 50  0001 C CNN
@@
 P 3600 4150
 AR Path="/6001D3BA" Ref="#PWR?"  Part="1"
-AR Path="/6017800E/6001D3BA" Ref="#PWR?"  Part="1"
-F 0 "#PWR?" H 3600 3900 50  0001 C CNN
+AR Path="/6017800E/6001D3BA" Ref="#PWR065"  Part="1"
+F 0 "#PWR065" H 3600 3900 50  0001 C CNN
 F 1 "GND" H 3605 3977 50  0000 C CNN
 F 2 "" H 3600 4150 50  0001 C CNN
@@
 P 4700 4150
 AR Path="/60039E54" Ref="C?"  Part="1"
-AR Path="/6017800E/60039E54" Ref="C?"  Part="1"
-F 0 "C?" H 4800 4150 50  0000 L CNN
+AR Path="/6017800E/60039E54" Ref="C41"  Part="1"
+F 0 "C41" H 4800 4150 50  0000 L CNN
 F 1 "0.1uF" H 4775 4075 50  0000 L CNN
 F 2 "" H 4700 4150 50  0001 C CNN
@@
 P 4800 4250
 AR Path="/6003A4FF" Ref="R?"  Part="1"
-AR Path="/6017800E/6003A4FF" Ref="R?"  Part="1"
-F 0 "R?" V 5000 4250 50  0000 C CNN
+AR Path="/6017800E/6003A4FF" Ref="R36"  Part="1"
+F 0 "R36" V 5000 4250 50  0000 C CNN
 F 1 "100" V 4900 4250 50  0000 C CNN
 F 2 "" H 4800 4250 50  0001 C CNN
@@
 P 4600 4150
 AR Path="/6003D903" Ref="#PWR?"  Part="1"
-AR Path="/6017800E/6003D903" Ref="#PWR?"  Part="1"
-F 0 "#PWR?" H 4600 3900 50  0001 C CNN
+AR Path="/6017800E/6003D903" Ref="#PWR068"  Part="1"
+F 0 "#PWR068" H 4600 3900 50  0001 C CNN
 F 1 "GND" H 4605 3977 50  0000 C CNN
 F 2 "" H 4600 4150 50  0001 C CNN
@@
 P 4300 4050
 AR Path="/600493FC" Ref="C?"  Part="1"
-AR Path="/6017800E/600493FC" Ref="C?"  Part="1"
-F 0 "C?" V 4525 3975 50  0000 L CNN
+AR Path="/6017800E/600493FC" Ref="C38"  Part="1"
+F 0 "C38" V 4525 3975 50  0000 L CNN
 F 1 "0.1uF" V 4450 3850 50  0000 L CNN
 F 2 "" H 4300 4050 50  0001 C CNN
@@
 	3100 4500 3100 4850
 Text Label 6500 3400 2    50   ~ 0
-VSS
+CBI
 Text Label 4750 3400 0    50   ~ 0
-VSS
+CBI
 Wire Wire Line
 	5850 3400 6500 3400
