File: uHoubolt_PCB_PMU/balancer.sch (KiCad schematic (older format))
At the start: 30 parts, among them Q3 BUK7M27-80EX, Q4 BUK7M27-80EX, U9 BQ77915

Commit message: small fix balancer schematic
Connections:
- net labels removed: CBI
Changed lines of the file:
@@
 $Descr A4 11693 8268
 encoding utf-8
-Sheet 4 5
+Sheet 5 5
 Title ""
 Date ""
@@
 Wire Wire Line
 	4100 2900 3700 2900
+Text HLabel 3300 3300 0    50   Input ~ 0
+BATT3V6
 Text HLabel 3350 3100 0    50   Input ~ 0
-BATT3V6
-Text HLabel 3300 3300 0    50   Input ~ 0
 BATT7V2
 Wire Wire Line
@@
 Wire Wire Line
 	3100 4500 3100 4850
-Text Label 6500 3400 2    50   ~ 0
-CBI
-Text Label 4750 3400 0    50   ~ 0
-CBI
-Wire Wire Line
-	5850 3400 6500 3400
+Wire Wire Line
+	5850 3400 6000 3400
 Wire Wire Line
 	6200 4125 6250 4125
@@
 Wire Wire Line
 	6050 3300 6125 3300
+$Comp
+L power:GND #PWR?
+U 1 1 5FF67558
+P 6000 3400
+AR Path="/5FF67558" Ref="#PWR?"  Part="1"
+AR Path="/6017800E/5FF67558" Ref="#PWR?"  Part="1"
+F 0 "#PWR?" H 6000 3150 50  0001 C CNN
+F 1 "GND" H 6005 3227 50  0000 C CNN
+F 2 "" H 6000 3400 50  0001 C CNN
+F 3 "" H 6000 3400 50  0001 C CNN
+	1    6000 3400
+	1    0    0    -1
+$EndComp
+$Comp
+L power:GND #PWR?
+U 1 1 5FF67769
+P 4750 3400
+AR Path="/5FF67769" Ref="#PWR?"  Part="1"
+AR Path="/6017800E/5FF67769" Ref="#PWR?"  Part="1"
+F 0 "#PWR?" H 4750 3150 50  0001 C CNN
+F 1 "GND" H 4755 3227 50  0000 C CNN
+F 2 "" H 4750 3400 50  0001 C CNN
+F 3 "" H 4750 3400 50  0001 C CNN
+	1    4750 3400
+	1    0    0    -1
+$EndComp
 $EndSCHEMATC

Commit message: bat+ lable change, change mosfets balancer, remove sys_load
Parts:
- removed Q3, Q4: BUK7M27-80EX, Package_TO_SOT_SMD:LFPAK33, symbol Transistor_FET:BUK7M27-80EX
- added Q? (x2): CSD17303Q5, Package_TO_SOT_SMD:TDSON-8-1, symbol Transistor_FET:CSD17303Q5
Changed lines of the file:
@@
 Comment4 ""
 $EndDescr
-$Comp
-L Transistor_FET:BUK7M27-80EX Q?
-U 1 1 601B6EBB
-P 6150 4400
-AR Path="/601B6EBB" Ref="Q?"  Part="1"
-AR Path="/6017800E/601B6EBB" Ref="Q4"  Part="1"
-F 0 "Q4" V 6350 4250 50  0000 L CNN
-F 1 "BUK7M27-80EX" V 6450 4000 50  0000 L CNN
-F 2 "Package_TO_SOT_SMD:LFPAK33" H 6350 4325 50  0001 L CIN
-F 3 "https://assets.nexperia.com/documents/data-sheet/BUK7M27-80E.pdf" V 6150 4400 50  0001 L CNN
-	1    6150 4400
-	0    -1   1    0
-$EndComp
 Connection ~ 4200 2500
 Wire Wire Line
@@
 Wire Wire Line
 	5500 3900 5750 3900
-$Comp
-L Transistor_FET:BUK7M27-80EX Q?
-U 1 1 601B6EDA
-P 5550 4400
-AR Path="/601B6EDA" Ref="Q?"  Part="1"
-AR Path="/6017800E/601B6EDA" Ref="Q3"  Part="1"
-F 0 "Q3" V 5750 4250 50  0000 L CNN
-F 1 "BUK7M27-80EX" V 5850 4050 50  0000 L CNN
-F 2 "Package_TO_SOT_SMD:LFPAK33" H 5750 4325 50  0001 L CIN
-F 3 "https://assets.nexperia.com/documents/data-sheet/BUK7M27-80E.pdf" V 5550 4400 50  0001 L CNN
-	1    5550 4400
-	0    1    1    0
-$EndComp
 Wire Wire Line
 	6850 3600 6850 4350
@@
 	1    0    0    -1
 $EndComp
+$Comp
+L Transistor_FET:CSD17303Q5 Q?
+U 1 1 5FFDCFF3
+P 5550 4400
+F 0 "Q?" V 5799 4400 50  0000 C CNN
+F 1 "CSD17303Q5" V 5890 4400 50  0000 C CNN
+F 2 "Package_TO_SOT_SMD:TDSON-8-1" H 5750 4325 50  0001 L CIN
+F 3 "http://www.ti.com/lit/gpn/csd17303q5" V 5550 4400 50  0001 L CNN
+	1    5550 4400
+	0    1    1    0
+$EndComp
+$Comp
+L Transistor_FET:CSD17303Q5 Q?
+U 1 1 5FFE07CF
+P 6150 4400
+F 0 "Q?" V 6399 4400 50  0000 C CNN
+F 1 "CSD17303Q5" V 6490 4400 50  0000 C CNN
+F 2 "Package_TO_SOT_SMD:TDSON-8-1" H 6350 4325 50  0001 L CIN
+F 3 "http://www.ti.com/lit/gpn/csd17303q5" V 6150 4400 50  0001 L CNN
+	1    6150 4400
+	0    1    1    0
+$EndComp
 $EndSCHEMATC

Commit message: Add descriptions
Parts:
- gave numbers to parts that had none: 2
Changed lines of the file:
@@
 $Descr A4 11693 8268
 encoding utf-8
-Sheet 5 5
+Sheet 2 4
 Title ""
 Date ""
@@
 P 6000 3400
 AR Path="/5FF67558" Ref="#PWR?"  Part="1"
-AR Path="/6017800E/5FF67558" Ref="#PWR?"  Part="1"
-F 0 "#PWR?" H 6000 3150 50  0001 C CNN
-F 1 "GND" H 6005 3227 50  0000 C CNN
+AR Path="/6017800E/5FF67558" Ref="#PWR072"  Part="1"
+F 0 "#PWR072" H 6000 3150 50  0001 C CNN
+F 1 "GND" H 6000 3250 50  0000 C CNN
 F 2 "" H 6000 3400 50  0001 C CNN
 F 3 "" H 6000 3400 50  0001 C CNN
@@
 P 4750 3400
 AR Path="/5FF67769" Ref="#PWR?"  Part="1"
-AR Path="/6017800E/5FF67769" Ref="#PWR?"  Part="1"
-F 0 "#PWR?" H 4750 3150 50  0001 C CNN
+AR Path="/6017800E/5FF67769" Ref="#PWR013"  Part="1"
+F 0 "#PWR013" H 4750 3150 50  0001 C CNN
 F 1 "GND" H 4755 3227 50  0000 C CNN
 F 2 "" H 4750 3400 50  0001 C CNN
@@
 $EndComp
 $Comp
-L Transistor_FET:CSD17303Q5 Q?
+L Transistor_FET:CSD17303Q5 Q3
 U 1 1 5FFDCFF3
 P 5550 4400
-F 0 "Q?" V 5799 4400 50  0000 C CNN
+F 0 "Q3" V 5799 4400 50  0000 C CNN
 F 1 "CSD17303Q5" V 5890 4400 50  0000 C CNN
 F 2 "Package_TO_SOT_SMD:TDSON-8-1" H 5750 4325 50  0001 L CIN
@@
 $EndComp
 $Comp
-L Transistor_FET:CSD17303Q5 Q?
+L Transistor_FET:CSD17303Q5 Q4
 U 1 1 5FFE07CF
 P 6150 4400
-F 0 "Q?" V 6399 4400 50  0000 C CNN
+F 0 "Q4" V 6399 4400 50  0000 C CNN
 F 1 "CSD17303Q5" V 6490 4400 50  0000 C CNN
 F 2 "Package_TO_SOT_SMD:TDSON-8-1" H 6350 4325 50  0001 L CIN

Commit message: unify notation, connect NoConnects, revise balancer, add output connector
Parts:
- C14: renamed from C34; value 0.1uF -> 100n
- C15: renamed from C35; value 1uF -> 1u
- C16: renamed from C36; value 1uF -> 1u
- C17: renamed from C37; value 1uF -> 1u
- C18: renamed from C38; value 0.1uF -> 100n
- C19: renamed from C39; value 1uF -> 1u
- C20: renamed from C40; value 1uF -> 1u
- C21: renamed from C41; value 0.1uF -> 100n
- C22: renamed from C42; value 1uF -> 1u
- renumbered D6 to D3, R29 to R20, R30 to R21, R31 to R22, R32 to R23, R33 to R24, R34 to R25, R35 to R26, R36 to R27, R37 to R28, R38 to R29, R39 to R30, R40 to R31, R41 to R32, R42 to R33, R43 to R34, R44 to R35, U9 to U3
Connections:
- net labels added: B_GND, GND_OUT
- net labels removed: GND
- wire segments 97 -> 103

Commit message: add NoConnects, add capacitor footprints, add pulldown to Q1
Parts:
- C14, C18, C21: footprint (none) -> Capacitor_SMD:C_0402_1005Metric
- C15, C16, C17, C19, C20, C22: footprint (none) -> Capacitor_SMD:C_0603_1608Metric
Changed lines of the file:
@@
 F 0 "C22" V 4850 2500 50  0000 L CNN
 F 1 "1u" V 4950 2500 50  0000 L CNN
-F 2 "" H 4800 2700 50  0001 C CNN
+F 2 "Capacitor_SMD:C_0603_1608Metric" H 4800 2700 50  0001 C CNN
 F 3 "~" H 4800 2700 50  0001 C CNN
 	1    4800 2700
@@
 F 0 "C20" H 4492 3646 50  0000 L CNN
 F 1 "1u" H 4492 3555 50  0000 L CNN
-F 2 "" H 4400 3600 50  0001 C CNN
+F 2 "Capacitor_SMD:C_0603_1608Metric" H 4400 3600 50  0001 C CNN
 F 3 "~" H 4400 3600 50  0001 C CNN
 	1    4400 3600
@@
 F 0 "C19" H 4492 3446 50  0000 L CNN
 F 1 "1u" H 4492 3355 50  0000 L CNN
-F 2 "" H 4400 3400 50  0001 C CNN
+F 2 "Capacitor_SMD:C_0603_1608Metric" H 4400 3400 50  0001 C CNN
 F 3 "~" H 4400 3400 50  0001 C CNN
 	1    4400 3400
@@
 F 0 "C15" H 4242 3246 50  0000 L CNN
 F 1 "1u" H 4242 3155 50  0000 L CNN
-F 2 "" H 4150 3200 50  0001 C CNN
+F 2 "Capacitor_SMD:C_0603_1608Metric" H 4150 3200 50  0001 C CNN
 F 3 "~" H 4150 3200 50  0001 C CNN
 	1    4150 3200
@@
 F 0 "C17" H 4392 3046 50  0000 L CNN
 F 1 "1u" H 4392 2955 50  0000 L CNN
-F 2 "" H 4300 3000 50  0001 C CNN
+F 2 "Capacitor_SMD:C_0603_1608Metric" H 4300 3000 50  0001 C CNN
 F 3 "~" H 4300 3000 50  0001 C CNN
 	1    4300 3000
@@
 F 0 "C16" H 4292 2446 50  0000 L CNN
 F 1 "1u" H 4292 2355 50  0000 L CNN
-F 2 "" H 4200 2400 50  0001 C CNN
+F 2 "Capacitor_SMD:C_0603_1608Metric" H 4200 2400 50  0001 C CNN
 F 3 "~" H 4200 2400 50  0001 C CNN
 	1    4200 2400
@@
 F 0 "C14" H 3792 4196 50  0000 L CNN
 F 1 "100n" H 3792 4105 50  0000 L CNN
-F 2 "" H 3700 4150 50  0001 C CNN
+F 2 "Capacitor_SMD:C_0402_1005Metric" H 3700 4150 50  0001 C CNN
 F 3 "~" H 3700 4150 50  0001 C CNN
 	1    3700 4150
@@
 F 0 "C21" H 4800 4150 50  0000 L CNN
 F 1 "100n" H 4775 4075 50  0000 L CNN
-F 2 "" H 4700 4150 50  0001 C CNN
+F 2 "Capacitor_SMD:C_0402_1005Metric" H 4700 4150 50  0001 C CNN
 F 3 "~" H 4700 4150 50  0001 C CNN
 	1    4700 4150
@@
 F 0 "C18" V 4525 3975 50  0000 L CNN
 F 1 "100n" V 4450 3850 50  0000 L CNN
-F 2 "" H 4300 4050 50  0001 C CNN
+F 2 "Capacitor_SMD:C_0402_1005Metric" H 4300 4050 50  0001 C CNN
 F 3 "~" H 4300 4050 50  0001 C CNN
 	1    4300 4050

Commit message: connect power flags, update main
Parts:
- R20, R21, R22, R23, R24, R25, R27, R28, R29, R30, R31, R32, R33, R34, R35: footprint (none) -> Resistor_SMD:R_0603_1608Metric
Changed lines of the file:
@@
 F 0 "R34" H 6400 3900 50  0000 R CNN
 F 1 "3.3M" H 6400 4000 50  0000 R CNN
-F 2 "" H 6450 3800 50  0001 C CNN
+F 2 "Resistor_SMD:R_0603_1608Metric" H 6450 3800 50  0001 C CNN
 F 3 "~" H 6450 3800 50  0001 C CNN
 	1    6450 3800
@@
 F 0 "R33" V 6225 3600 50  0000 C CNN
 F 1 "1M" V 6150 3575 50  0000 C CNN
-F 2 "" H 6100 3700 50  0001 C CNN
+F 2 "Resistor_SMD:R_0603_1608Metric" H 6100 3700 50  0001 C CNN
 F 3 "~" H 6100 3700 50  0001 C CNN
 	1    6100 3700
@@
 F 0 "R35" V 6800 3600 50  0000 C CNN
 F 1 "470k" V 6900 3650 50  0000 C CNN
-F 2 "" H 6700 3600 50  0001 C CNN
+F 2 "Resistor_SMD:R_0603_1608Metric" H 6700 3600 50  0001 C CNN
 F 3 "~" H 6700 3600 50  0001 C CNN
 	1    6700 3600
@@
 F 0 "R29" H 5400 3950 50  0000 R CNN
 F 1 "1M" H 5441 4045 50  0000 R CNN
-F 2 "" H 5500 4000 50  0001 C CNN
+F 2 "Resistor_SMD:R_0603_1608Metric" H 5500 4000 50  0001 C CNN
 F 3 "~" H 5500 4000 50  0001 C CNN
 	1    5500 4000
@@
 F 0 "R28" V 5450 3850 50  0000 C CNN
 F 1 "4.5k" V 5550 3800 50  0000 C CNN
-F 2 "" H 5350 3900 50  0001 C CNN
+F 2 "Resistor_SMD:R_0603_1608Metric" H 5350 3900 50  0001 C CNN
 F 3 "~" H 5350 3900 50  0001 C CNN
 	1    5350 3900
@@
 F 0 "R30" V 6000 2650 50  0000 C CNN
 F 1 "10k" V 5900 2650 50  0000 C CNN
-F 2 "" H 5950 2800 50  0001 C CNN
+F 2 "Resistor_SMD:R_0603_1608Metric" H 5950 2800 50  0001 C CNN
 F 3 "~" H 5950 2800 50  0001 C CNN
 	1    5950 2800
@@
 F 0 "R32" V 5900 3450 50  0000 C CNN
 F 1 "100k" V 6000 3425 50  0000 C CNN
-F 2 "" H 5950 3300 50  0001 C CNN
+F 2 "Resistor_SMD:R_0603_1608Metric" H 5950 3300 50  0001 C CNN
 F 3 "~" H 5950 3300 50  0001 C CNN
 	1    5950 3300
@@
 F 0 "R31" V 5900 3250 50  0000 C CNN
 F 1 "10k" V 6000 3200 50  0000 C CNN
-F 2 "" H 5950 3100 50  0001 C CNN
+F 2 "Resistor_SMD:R_0603_1608Metric" H 5950 3100 50  0001 C CNN
 F 3 "~" H 5950 3100 50  0001 C CNN
 	1    5950 3100
@@
 F 0 "R23" V 3854 3750 50  0000 C CNN
 F 1 "134" V 3945 3750 50  0000 C CNN
-F 2 "" H 4050 3750 50  0001 C CNN
+F 2 "Resistor_SMD:R_0603_1608Metric" H 4050 3750 50  0001 C CNN
 F 3 "~" H 4050 3750 50  0001 C CNN
 	1    4050 3750
@@
 F 0 "R22" V 4100 3150 50  0000 C CNN
 F 1 "134" V 4200 3150 50  0000 C CNN
-F 2 "" H 4050 3300 50  0001 C CNN
+F 2 "Resistor_SMD:R_0603_1608Metric" H 4050 3300 50  0001 C CNN
 F 3 "~" H 4050 3300 50  0001 C CNN
 	1    4050 3300
@@
 F 0 "R20" V 3900 2950 50  0000 C CNN
 F 1 "134" V 4000 2950 50  0000 C CNN
-F 2 "" H 3850 3100 50  0001 C CNN
+F 2 "Resistor_SMD:R_0603_1608Metric" H 3850 3100 50  0001 C CNN
 F 3 "~" H 3850 3100 50  0001 C CNN
 	1    3850 3100
@@
 F 0 "R24" V 4000 2850 50  0000 C CNN
 F 1 "134" V 4100 2850 50  0000 C CNN
-F 2 "" H 4200 2900 50  0001 C CNN
+F 2 "Resistor_SMD:R_0603_1608Metric" H 4200 2900 50  0001 C CNN
 F 3 "~" H 4200 2900 50  0001 C CNN
 	1    4200 2900
@@
 F 0 "R21" V 3754 2300 50  0000 C CNN
 F 1 "1k" V 3845 2300 50  0000 C CNN
-F 2 "" H 3950 2300 50  0001 C CNN
+F 2 "Resistor_SMD:R_0603_1608Metric" H 3950 2300 50  0001 C CNN
 F 3 "~" H 3950 2300 50  0001 C CNN
 	1    3950 2300
@@
 Wire Wire Line
 	6300 3700 6450 3700
-Text HLabel 3550 2300 0    50   Input ~ 0
-BATT_VCC
 Wire Wire Line
 	3550 2300 3850 2300
-Text HLabel 3700 2900 0    50   Input ~ 0
-BATT_VCC
 Wire Wire Line
 	4100 2900 3700 2900
-Text HLabel 3300 3300 0    50   Input ~ 0
-BATT3V6
-Text HLabel 3350 3100 0    50   Input ~ 0
-BATT7V2
 Wire Wire Line
 	3350 3100 3750 3100
@@
 F 0 "R25" V 4250 4000 50  0000 C CNN
 F 1 "100" V 4150 4000 50  0000 C CNN
-F 2 "" H 4200 4150 50  0001 C CNN
+F 2 "Resistor_SMD:R_0603_1608Metric" H 4200 4150 50  0001 C CNN
 F 3 "~" H 4200 4150 50  0001 C CNN
 	1    4200 4150
@@
 F 0 "R27" V 5000 4250 50  0000 C CNN
 F 1 "100" V 4900 4250 50  0000 C CNN
-F 2 "" H 4800 4250 50  0001 C CNN
+F 2 "Resistor_SMD:R_0603_1608Metric" H 4800 4250 50  0001 C CNN
 F 3 "~" H 4800 4250 50  0001 C CNN
 	1    4800 4250
@@
 Wire Wire Line
 	6850 3600 7350 3600
-Text HLabel 7350 3600 2    50   Input ~ 0
-GND_OUT
 Text Label 3375 4150 0    50   ~ 0
 B_GND
@@
 Wire Wire Line
 	6050 3300 6875 3300
+Text HLabel 3550 2300 0    50   Input ~ 0
+BATT_VCC
+Text HLabel 3700 2900 0    50   Input ~ 0
+BATT_VCC
+Text HLabel 3350 3100 0    50   Input ~ 0
+BATT7V2
+Text HLabel 3300 3300 0    50   Input ~ 0
+BATT3V6
+Text HLabel 7350 3600 2    50   Input ~ 0
+GND_OUT
 $EndSCHEMATC

Commit message: add mosfet in schematic, draw outer bounds of pcb
Parts:
- D3: footprint (none) -> Diode_SMD:D_SOT-23_ANK
- TH1: footprint (none) -> Resistor_SMD:R_0603_1608Metric
- U3: footprint (none) -> Package_SO:TSSOP-24_4.4x7.8mm_P0.65mm
Changed lines of the file:
@@
 Wire Wire Line
 	4900 2600 4700 2600
-Wire Wire Line
-	4050 2300 4200 2300
 $Comp
 L Device:R_Small R?
@@
 F 0 "U3" H 5375 3925 50  0000 C CNN
 F 1 "BQ77915" H 5375 3834 50  0000 C CNN
-F 2 "" H 5350 3250 50  0001 C CNN
+F 2 "Package_SO:TSSOP-24_4.4x7.8mm_P0.65mm" H 5350 3250 50  0001 C CNN
 F 3 "" H 5350 3250 50  0001 C CNN
 	1    5350 3150
@@
 Wire Wire Line
 	6300 3700 6450 3700
-Wire Wire Line
-	3550 2300 3850 2300
 Wire Wire Line
 	4100 2900 3700 2900
@@
 F 0 "TH1" V 6210 3200 50  0000 C CNN
 F 1 "Thermistor_NTC" V 6301 3200 50  0000 C CNN
-F 2 "" H 6500 3250 50  0001 C CNN
+F 2 "Resistor_SMD:R_0603_1608Metric" H 6500 3250 50  0001 C CNN
 F 3 "~" H 6500 3250 50  0001 C CNN
 	1    6500 3200
@@
 F 0 "D3" H 6050 3909 50  0000 C CNN
 F 1 "D_Zener" H 6050 4000 50  0000 C CNN
-F 2 "" H 6050 4125 50  0001 C CNN
+F 2 "Diode_SMD:D_SOT-23_ANK" H 6050 4125 50  0001 C CNN
 F 3 "~" H 6050 4125 50  0001 C CNN
 	1    6050 4125
@@
 Text HLabel 7350 3600 2    50   Input ~ 0
 GND_OUT
+$Comp
+L power:PWR_FLAG #FLG0105
+U 1 1 6094DFD4
+P 4200 2300
+F 0 "#FLG0105" H 4200 2375 50  0001 C CNN
+F 1 "PWR_FLAG" H 4325 2450 50  0000 C CNN
+F 2 "" H 4200 2300 50  0001 C CNN
+F 3 "~" H 4200 2300 50  0001 C CNN
+	1    4200 2300
+	1    0    0    -1
+$EndComp
+Wire Wire Line
+	3550 2300 3850 2300
+Wire Wire Line
+	4050 2300 4200 2300
 $EndSCHEMATC

Commit message: add ignition bus, placement 75% done
Parts:
- removed TH1: Thermistor_NTC, Resistor_SMD:R_0603_1608Metric, symbol Device:Thermistor_NTC
- added J_TH1: Conn_01x02_MP, Connector_JST:JST_GH_BM02B-GHS-TBT_1x02-1MP_P1.25mm_Vertical, symbol Connector_Generic_MountingPin:Conn_01x02_MountingPin
Connections:
- wire segments 103 -> 105
Changed lines of the file:
@@
 Connection ~ 6850 3600
 NoConn ~ 5850 2900
-$Comp
-L Device:Thermistor_NTC TH1
-U 1 1 5FF5E99E
-P 6500 3200
-F 0 "TH1" V 6210 3200 50  0000 C CNN
-F 1 "Thermistor_NTC" V 6301 3200 50  0000 C CNN
-F 2 "Resistor_SMD:R_0603_1608Metric" H 6500 3250 50  0001 C CNN
-F 3 "~" H 6500 3250 50  0001 C CNN
-	1    6500 3200
-	0    1    1    0
-$EndComp
-Wire Wire Line
-	6150 3200 6350 3200
 Connection ~ 6150 3200
-Wire Wire Line
-	6650 3200 7050 3200
 $Comp
 L Device:D_Zener D3
@@
 	6200 2850 7050 2850
 Wire Wire Line
-	7050 2850 7050 3200
+	7050 2850 7050 3000
 Connection ~ 7050 3200
 Wire Wire Line
@@
 Text Label 7450 3200 2    50   ~ 0
 B_GND
-Wire Wire Line
-	7050 3200 7450 3200
 Text Label 6875 3300 2    50   ~ 0
 B_GND
@@
 Wire Wire Line
 	4050 2300 4200 2300
+Wire Wire Line
+	6150 3200 6450 3200
+Wire Wire Line
+	6550 3200 7050 3200
+$Comp
+L Connector_Generic_MountingPin:Conn_01x02_MountingPin J_TH1
+U 1 1 607BBD1D
+P 6450 3000
+F 0 "J_TH1" V 6550 2925 50  0000 C CNN
+F 1 "Conn_01x02_MP" V 6550 2800 50  0001 C CNN
+F 2 "Connector_JST:JST_GH_BM02B-GHS-TBT_1x02-1MP_P1.25mm_Vertical" H 6450 3000 50  0001 C CNN
+F 3 "~" H 6450 3000 50  0001 C CNN
+	1    6450 3000
+	0    -1   -1   0
+$EndComp
+Wire Wire Line
+	7050 3200 7450 3200
+Wire Wire Line
+	6750 3000 7050 3000
+Connection ~ 7050 3000
+Wire Wire Line
+	7050 3000 7050 3200
 $EndSCHEMATC
