File: uHoubolt_PCB_PMU/uHoubolt_PCB_PMU.sch (KiCad schematic (older format))
At the start: 0 parts

Commit message: balancer connected
Parts:
- added C? (x2): C_Small, symbol Device:C_Small
- added J?: Conn_01x04, symbol Connector_Generic:Conn_01x04
- added J?: Conn_01x02, symbol Connector_Generic:Conn_01x02
- added R? (x3): 1k, symbol Device:R_Small
- added R? (x5): R_Small, symbol Device:R_Small
- added RV?: R_POT_Small, symbol Device:R_POT_Small
- added SW? (x2): SW_Push_SPDT, symbol Switch:SW_Push_SPDT
- added U?: BQ77915, symbol TXV_LIB:BQ77915
Connections:
- net labels added: BATT3V6, BATT7V2, BATT_GND, BATT_VCC, GND
- wire segments 0 -> 40
- no-connect marks 0 -> 5

Commit message: charge controller added
Parts:
- removed C?: C_Small, symbol Device:C_Small
- added C? (x2): 0.22u, symbol Device:C_Small
- added C?: 2.2u, symbol Device:C_Small
- added C? (x2): 0.01u, symbol Device:C_Small
- added C? (x2): 47n, symbol Device:C_Small
- added C?: 0.1u, symbol Device:C_Small
- added C? (x5): 1uF, symbol Device:C_Small
- added C?: 1n, symbol Device:C_Small
- added C?: 1u, symbol Device:C_Small
- added C?: 47u, symbol Device:CP1
- added C?: 68uF, symbol Device:CP1
- added D? (x2): D_Schottky, symbol Device:D_Schottky
- added L?: 10uH, symbol Device:L_Small
- added Q?: Si7141DP, Package_SO:PowerPAK_SO-8_Single, symbol Transistor_FET:Si7141DP
- added Q? (x3): BUK7M27-80EX, Package_TO_SOT_SMD:LFPAK33, symbol Transistor_FET:BUK7M27-80EX
- added R? (x2): 4.7, symbol Device:R_Small
- added R?: 100k, symbol Device:R_Small
- added R?: 10k, symbol Device:R_Small
- added R?: 0.033, symbol Device:R_Small
- added R? (x5): R_Small, symbol Device:R_Small
- added R? (x2): 1M, symbol Device:R_Small
- added R?: 470k, symbol Device:R_Small
- added R?: 0.068, symbol Device:R_Small
- added U?: MAX1873SEEE, Package_SO:QSOP-16_3.9x4.9mm_P0.635mm, symbol Battery_Management:MAX1873SEEE
- C?: value C_Small -> 1uF
- R? (x4): value R_Small -> 33
- R?: value 1k -> 10k
- R?: value 1k -> 100k
- R?: value R_Small -> 10k
- RV?: value R_POT_Small -> 10k
Connections:
- net labels added: DISABLE, IOUT, SYS_LOAD
- wire segments 40 -> 165
Other:
- moved on the sheet: C?, J?, R?, SW?, U?

Commit message: hierarchies, buck converters added
Parts:
- removed C? (x6): 1uF, symbol Device:C_Small
- removed Q? (x2): BUK7M27-80EX, Package_TO_SOT_SMD:LFPAK33, symbol Transistor_FET:BUK7M27-80EX
- removed R?: 1k, symbol Device:R_Small
- removed R? (x4): 33, symbol Device:R_Small
- removed R? (x2): 10k, symbol Device:R_Small
- removed R?: 100k, symbol Device:R_Small
- removed R? (x3): R_Small, symbol Device:R_Small
- removed R? (x2): 1M, symbol Device:R_Small
- removed R?: 470k, symbol Device:R_Small
- removed RV?: 10k, symbol Device:R_POT_Small
- removed U?: BQ77915, symbol TXV_LIB:BQ77915
- added C?: 22uF, Capacitor_SMD:C_0603_1608Metric, symbol Device:C_Small
- added U?: AMS1117-3.3, Package_TO_SOT_SMD:SOT-223-3_TabPin2, symbol Regulator_Linear:AMS1117-3.3
Connections:
- net labels added: VIN, VOUT
- wire segments 165 -> 101
- no-connect marks 5 -> 2
Other:
- moved on the sheet: Q?

Commit message: added CAN connector, current measurement and hierarchial labels
Parts:
- removed C?: 22uF, Capacitor_SMD:C_0603_1608Metric, symbol Device:C_Small
- removed U?: AMS1117-3.3, Package_TO_SOT_SMD:SOT-223-3_TabPin2, symbol Regulator_Linear:AMS1117-3.3
- added C1, C2: 100n, Capacitor_SMD:C_0603_1608Metric, symbol Device:C_Small
- added J3: Conn_01x04, symbol Connector_Generic:Conn_01x04
- added R1, R3, R5: 10k, symbol Device:R_Small
- added R11, R12, R8: 10k, Resistor_SMD:R_0603_1608Metric, symbol Device:R_Small
- added R2, R4: 2k, symbol Device:R_Small
- added R6: 1k, symbol Device:R_Small
- added U1: INA260, Package_SO:TSSOP-16_4.4x5mm_P0.65mm, symbol Sensor:INA260
- gave numbers to parts that had none: 30
Connections:
- net labels added: ALERT, CAN2_H, CAN2_L, CELL_3V6, CELL_7V2, CHARGE_VOLT, I2C_SCL, I2C_SDA, VCC
- net labels removed: +5V, VIN, VOUT
- wire segments 101 -> 137
Other:
- note added: "Addr: 0x40"

Commit message: add current measurement
Parts:
- removed C1, C2: 100n, Capacitor_SMD:C_0603_1608Metric, symbol Device:C_Small
- removed J3: Conn_01x04, symbol Connector_Generic:Conn_01x04
- removed R11, R12, R8: 10k, Resistor_SMD:R_0603_1608Metric, symbol Device:R_Small
- removed U1: INA260, Package_SO:TSSOP-16_4.4x5mm_P0.65mm, symbol Sensor:INA260
- added C?: 0.1u, symbol Device:C_Small
- added J?: Conn_01x04, symbol Connector_Generic:Conn_01x04
- added R? (x3): 2.7k, symbol Device:R_Small
- added R?: 4m, symbol Device:R_Small
- added U?: INA226, Package_SO:VSSOP-10_3x3mm_P0.5mm, symbol Analog_ADC:INA226
Connections:
- net labels added: CAN_H, CAN_L, SCL, SDA
- net labels removed: CAN2_H, CAN2_L
- wire segments 137 -> 146
Other:
- note added: "Adress: 0x40\n"
- note removed: "Addr: 0x40"

Commit message: add resistor values of regulator
Parts:
- R10, R9: value R_Small -> 100k
Connections:
- wire segments 146 -> 147
Other:
- moved on the sheet: C10, C11, C7, C9, R13, R?
Changed lines of the file:
@@
 U 1 1 5FDE89B3
 P 7900 3800
-F 0 "U2" H 7900 4581 50  0000 C CNN
-F 1 "MAX1873SEEE" H 7900 4490 50  0000 C CNN
+F 0 "U2" H 8025 4500 50  0000 C CNN
+F 1 "MAX1873SEEE" H 8175 4400 50  0000 C CNN
 F 2 "Package_SO:QSOP-16_3.9x4.9mm_P0.635mm" H 7900 3100 50  0001 C CNN
 F 3 "https://datasheets.maximintegrated.com/en/ds/MAX1873.pdf" H 8100 3800 50  0001 C CNN
@@
 P 6700 3900
 F 0 "R9" H 6800 3900 50  0000 L CNN
-F 1 "R_Small" H 6750 3800 50  0000 L CNN
+F 1 "100k" H 6750 3800 50  0000 L CNN
 F 2 "" H 6700 3900 50  0001 C CNN
 F 3 "~" H 6700 3900 50  0001 C CNN
@@
 L Device:C_Small C9
 U 1 1 5FE11561
-P 8850 4800
-F 0 "C9" V 8621 4800 50  0000 C CNN
-F 1 "47n" V 8712 4800 50  0000 C CNN
-F 2 "" H 8850 4800 50  0001 C CNN
-F 3 "~" H 8850 4800 50  0001 C CNN
-	1    8850 4800
+P 8850 4850
+F 0 "C9" V 8621 4850 50  0000 C CNN
+F 1 "47n" V 8712 4850 50  0000 C CNN
+F 2 "" H 8850 4850 50  0001 C CNN
+F 3 "~" H 8850 4850 50  0001 C CNN
+	1    8850 4850
 	0    1    1    0
 $EndComp
@@
 L Device:C_Small C10
 U 1 1 5FE1595A
-P 8850 5100
-F 0 "C10" V 8650 5100 50  0000 C CNN
-F 1 "47n" V 8712 5100 50  0000 C CNN
-F 2 "" H 8850 5100 50  0001 C CNN
-F 3 "~" H 8850 5100 50  0001 C CNN
-	1    8850 5100
+P 8850 5225
+F 0 "C10" V 8650 5225 50  0000 C CNN
+F 1 "47n" V 8750 5225 50  0000 C CNN
+F 2 "" H 8850 5225 50  0001 C CNN
+F 3 "~" H 8850 5225 50  0001 C CNN
+	1    8850 5225
 	0    1    1    0
 $EndComp
@@
 L Device:C_Small C11
 U 1 1 5FE163B6
-P 8850 5350
-F 0 "C11" V 8621 5350 50  0000 C CNN
-F 1 "0.1u" V 8750 5300 50  0000 C CNN
-F 2 "" H 8850 5350 50  0001 C CNN
-F 3 "~" H 8850 5350 50  0001 C CNN
-	1    8850 5350
+P 8850 5575
+F 0 "C11" V 8650 5525 50  0000 C CNN
+F 1 "0.1u" V 8750 5525 50  0000 C CNN
+F 2 "" H 8850 5575 50  0001 C CNN
+F 3 "~" H 8850 5575 50  0001 C CNN
+	1    8850 5575
 	0    1    1    0
 $EndComp
 Wire Wire Line
-	8650 5350 8750 5350
-Wire Wire Line
-	8950 5350 8950 5100
-Wire Wire Line
-	8950 4800 8950 5100
-Connection ~ 8950 5100
+	8650 5575 8750 5575
+Wire Wire Line
+	8950 5575 8950 5225
+Wire Wire Line
+	8950 4850 8950 5225
+Connection ~ 8950 5225
 $Comp
 L Device:C_Small C7
 U 1 1 5FE259AF
-P 8400 5600
-F 0 "C7" V 8550 5600 50  0000 C CNN
-F 1 "1n" V 8650 5600 50  0000 C CNN
-F 2 "" H 8400 5600 50  0001 C CNN
-F 3 "~" H 8400 5600 50  0001 C CNN
-	1    8400 5600
+P 8400 5775
+F 0 "C7" V 8550 5775 50  0000 C CNN
+F 1 "1n" V 8650 5775 50  0000 C CNN
+F 2 "" H 8400 5775 50  0001 C CNN
+F 3 "~" H 8400 5775 50  0001 C CNN
+	1    8400 5775
 	0    1    1    0
 $EndComp
 Wire Wire Line
-	8400 5100 8750 5100
-Wire Wire Line
-	8500 4800 8750 4800
-Wire Wire Line
-	8500 5600 8950 5600
-Wire Wire Line
-	8950 5600 8950 5350
-Connection ~ 8950 5350
+	8400 5225 8750 5225
+Wire Wire Line
+	8500 4850 8750 4850
+Wire Wire Line
+	8500 5775 8950 5775
+Wire Wire Line
+	8950 5775 8950 5575
+Connection ~ 8950 5575
 $Comp
 L power:GND #PWR0105
 U 1 1 5FE3A383
-P 8950 5600
-F 0 "#PWR0105" H 8950 5350 50  0001 C CNN
-F 1 "GND" H 8955 5427 50  0000 C CNN
-F 2 "" H 8950 5600 50  0001 C CNN
-F 3 "" H 8950 5600 50  0001 C CNN
-	1    8950 5600
-	1    0    0    -1
-$EndComp
-Connection ~ 8950 5600
+P 8950 5775
+F 0 "#PWR0105" H 8950 5525 50  0001 C CNN
+F 1 "GND" H 8955 5602 50  0000 C CNN
+F 2 "" H 8950 5775 50  0001 C CNN
+F 3 "" H 8950 5775 50  0001 C CNN
+	1    8950 5775
+	1    0    0    -1
+$EndComp
+Connection ~ 8950 5775
 $Comp
 L Device:R_Small R10
@@
 P 6700 4600
 F 0 "R10" H 6759 4646 50  0000 L CNN
-F 1 "R_Small" H 6759 4555 50  0000 L CNN
+F 1 "100k" H 6759 4555 50  0000 L CNN
 F 2 "" H 6700 4600 50  0001 C CNN
 F 3 "~" H 6700 4600 50  0001 C CNN
@@
 U 1 1 5FDF02D6
 P 7500 4100
-F 0 "C5" V 7300 4100 50  0000 C CNN
-F 1 "2.2u" V 7400 4100 50  0000 C CNN
+F 0 "C5" H 7375 4100 50  0000 C CNN
+F 1 "2.2u" H 7375 4000 50  0000 C CNN
 F 2 "" H 7500 4100 50  0001 C CNN
 F 3 "~" H 7500 4100 50  0001 C CNN
@@
 U 1 1 5FECF12C
 P 9950 4650
-F 0 "R17" H 10009 4696 50  0000 L CNN
-F 1 "0.068" H 10009 4605 50  0000 L CNN
+F 0 "R17" V 10025 4575 50  0000 L CNN
+F 1 "0.068" V 10100 4525 50  0000 L CNN
 F 2 "" H 9950 4650 50  0001 C CNN
 F 3 "~" H 9950 4650 50  0001 C CNN
@@
 P 6050 4050
 F 0 "#PWR0112" H 6050 3800 50  0001 C CNN
-F 1 "GND" V 6055 3922 50  0000 R CNN
+F 1 "GND" H 6125 3875 50  0000 R CNN
 F 2 "" H 6050 4050 50  0001 C CNN
 F 3 "" H 6050 4050 50  0001 C CNN
@@
 	1    0    0    -1
 $EndComp
-Connection ~ 8300 5350
-Wire Wire Line
-	8300 5350 8300 5600
-Wire Wire Line
-	8300 5350 8450 5350
 $Comp
 L Device:R_Small R13
 U 1 1 5FE16F9A
-P 8550 5350
-F 0 "R13" V 8350 5300 50  0000 L CNN
-F 1 "10k" V 8450 5300 50  0000 L CNN
-F 2 "" H 8550 5350 50  0001 C CNN
-F 3 "~" H 8550 5350 50  0001 C CNN
-	1    8550 5350
+P 8550 5575
+F 0 "R13" V 8350 5525 50  0000 L CNN
+F 1 "10k" V 8450 5525 50  0000 L CNN
+F 2 "" H 8550 5575 50  0001 C CNN
+F 3 "~" H 8550 5575 50  0001 C CNN
+	1    8550 5575
 	0    1    1    0
 $EndComp
@@
 	7100 2600 9550 2600
 Wire Wire Line
-	8300 4200 8300 5350
-Wire Wire Line
 	8300 4100 8400 4100
 Wire Wire Line
-	8400 4100 8400 5100
+	8400 4100 8400 5225
 Wire Wire Line
 	8300 4000 8500 4000
 Wire Wire Line
-	8500 4000 8500 4800
+	8500 4000 8500 4850
 Wire Wire Line
 	8300 3900 8600 3900
@@
 L Device:R_Small R?
 U 1 1 600E58A6
-P 4850 1800
-F 0 "R?" H 4650 1800 50  0000 L CNN
-F 1 "4m" H 4625 1725 50  0000 L CNN
-F 2 "" H 4850 1800 50  0001 C CNN
-F 3 "~" H 4850 1800 50  0001 C CNN
-	1    4850 1800
+P 4850 1750
+F 0 "R?" H 4650 1750 50  0000 L CNN
+F 1 "4m" H 4625 1675 50  0000 L CNN
+F 2 "" H 4850 1750 50  0001 C CNN
+F 3 "~" H 4850 1750 50  0001 C CNN
+	1    4850 1750
 	1    0    0    -1
 $EndComp
@@
 $EndComp
 Wire Wire Line
-	5550 1700 5550 1650
-Wire Wire Line
 	6800 1050 7150 1050
 Wire Wire Line
@@
 $EndComp
 Wire Wire Line
-	4850 1900 4850 2125
-Wire Wire Line
-	5550 1900 5550 1750
-Connection ~ 4850 1900
+	4850 1850 4850 2075
+Connection ~ 4850 1850
 Text Label 6650 1850 2    50   ~ 0
-ALERT
-Text Label 4000 4550 2    50   ~ 0
 ALERT
 Text Label 6550 1550 2    50   ~ 0
@@
 Text Notes 6300 1150 0    50   ~ 0
 Adress: 0x40\n
-Wire Wire Line
-	4850 1700 5250 1700
 $Comp
 L Connector_Generic:Conn_01x04 J?
@@
 L power:+BATT #PWR?
 U 1 1 60315C09
-P 4850 2125
-F 0 "#PWR?" H 4850 1975 50  0001 C CNN
-F 1 "+BATT" V 4865 2252 50  0000 L CNN
-F 2 "" H 4850 2125 50  0001 C CNN
-F 3 "" H 4850 2125 50  0001 C CNN
-	1    4850 2125
+P 4850 2075
+F 0 "#PWR?" H 4850 1925 50  0001 C CNN
+F 1 "+BATT" V 4865 2202 50  0000 L CNN
+F 2 "" H 4850 2075 50  0001 C CNN
+F 3 "" H 4850 2075 50  0001 C CNN
+	1    4850 2075
 	0    -1   -1   0
 $EndComp
 Wire Wire Line
-	4850 1900 5550 1900
+	4850 1850 5550 1850
 Wire Wire Line
 	5550 1250 5250 1250
-Wire Wire Line
-	5250 1250 5250 1700
-Connection ~ 5250 1700
-Wire Wire Line
-	5250 1700 5550 1700
 $Comp
 L power:GND #PWR?
@@
 Wire Wire Line
 	925  4175 1600 4175
-Text Label 4875 1700 0    50   ~ 0
+Text Label 4875 1650 0    50   ~ 0
 BATT_VCC
+Text Label 3400 5250 2    50   ~ 0
+IOUT
+Wire Wire Line
+	8300 4200 8300 5575
+Wire Wire Line
+	8450 5575 8300 5575
+Connection ~ 8300 5575
+Wire Wire Line
+	8300 5575 8300 5775
+Wire Wire Line
+	3000 5250 3400 5250
+Text Label 3400 5350 2    50   ~ 0
+ALERT
+Wire Wire Line
+	3000 5350 3400 5350
+Wire Wire Line
+	4850 1650 5250 1650
+Wire Wire Line
+	5550 1750 5550 1850
+Wire Wire Line
+	5250 1250 5250 1650
+Connection ~ 5250 1650
+Wire Wire Line
+	5250 1650 5550 1650
 $EndSCHEMATC

Commit message: connect labels to muC
Parts:
- gave numbers to parts that had none: 7
- renumbered C11 to C10, C12 to C11, C13 to C12, C14 to C13, C3 to C2, C4 to C3, C5 to C4, C6 to C5, C7 to C6, C8 to C7, C9 to C8, C10 to C9, R13 to R14, R14 to R15, R15 to R16, R16 to R17, R17 to R18, R7 to R8
Connections:
- wire segments 147 -> 149
