File: uHoubolt_PCB_PMU/uHoubolt_PCB_PMU.kicad_pcb (KiCad board)
At the start: 4 copper layers, 128 parts, among them J1 Conn_01x04, J2 Conn_01x02, J3 Conn_01x04_MountingPin, J4 Conn_01x02, J5 Conn_02x04_Odd_Even, J6 Conn_01x04_MountingPin, J7 Conn_01x04_MountingPin, J8 Conn_01x04_MountingPin, J9 Conn_01x04_MountingPin, Q1 ZXMN3F30FH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

Commit message: add ignition bus, placement 75% done
Parts:
- removed J2: Conn_01x02, Connector_Molex:Molex_PicoBlade_53047-0210_1x02_P1.25mm_Vertical
- removed the Q5 at (271.4, -14.8)
- removed the Q5 at (352.3, 9.53)
- removed the Q6 at (362.1, 3.68)
- removed TH1: Thermistor_NTC, Resistor_SMD:R_0603_1608Metric
- added C47: 100n, Capacitor_SMD:C_0402_1005Metric, F.Cu at (219.9, 159.8)
- added J10: Conn_01x02, Connector_Molex:Molex_Micro-Fit_3.0_43650-0215_1x02_P3.00mm_Vertical, F.Cu at (101.6, 93.0)
- added J_OUT1: Conn_01x02, Connector_Molex:Molex_Mega-Fit_76829-0002_2x01_P5.70mm_Vertical, F.Cu at (109.6, 90.6)
- added J_TH1: Conn_01x02_MP, Connector_JST:JST_GH_BM02B-GHS-TBT_1x02-1MP_P1.25mm_Vertical, F.Cu at (199.2, 89.8)
- added Q5: MMBT3904, Package_TO_SOT_SMD:SOT-23, F.Cu at (115.2, 100.7)
- added Q7: MMBT3904, Package_TO_SOT_SMD:SOT-23, F.Cu at (117.6, 80.0)
- added Q8: Si7141DP, Package_SO:PowerPAK_SO-8_Single, F.Cu at (110.4, 76.8)
- added Q9: BSF030NE2LQ, Package_DirectFET:DirectFET_SQ, F.Cu at (108.0, 83.4)
- added R49: 1k, Resistor_SMD:R_0603_1608Metric, F.Cu at (115.0, 80.2)
- added R50: 1k, Resistor_SMD:R_0603_1608Metric, F.Cu at (224.5, 158.6)
- added R52: 2.7k, Resistor_SMD:R_0603_1608Metric, F.Cu at (130.7, 105.6)
- added R53: 2.7k, Resistor_SMD:R_0603_1608Metric, F.Cu at (228.5, 158.6)
- added R54: 2.7k, Resistor_SMD:R_0603_1608Metric, F.Cu at (135.7, 94.2)
- added R55: 1k, Resistor_SMD:R_0603_1608Metric, F.Cu at (135.7, 96.7)
- added SW2: SW_Push_SPDT, TXV_LIB:MicroSwitch, F.Cu at (120.2, 73.4)
- added U10: INA226, Package_SO:VSSOP-10_3x3mm_P0.5mm, F.Cu at (214.8, 158.5)
- C34, C43, C44, C45, C46, J5, J6, J7, J8, J9, R42: moved to B.Cu
- J_BALANCE1: renamed from J1; footprint Connector_Molex:Molex_PicoBlade_53048-0410_1x04_P1.25mm_Horizontal -> Connector_JST:JST_XH_B4B-XH-AM_1x04_P2.50mm_Vertical
- J_IN1: renamed from J4; footprint Connector_Molex:Molex_PicoBlade_53048-0210_1x02_P1.25mm_Horizontal -> Connector_Molex:Molex_Mega-Fit_76829-0002_2x01_P5.70mm_Vertical
- J_UMBILICAL1: renamed from J3; footprint Connector_JST:JST_GH_SM04B-GHS-TB_1x04-1MP_P1.25mm_Horizontal -> Connector_Molex:Molex_MicroClasp_55932-0510_1x05_P2.00mm_Vertical
- moved J_IN1 302.4 mm to (102.2, 113.8)
- moved C39 295.9 mm to (109.2, 135.2), turned to 180 degrees
- moved U9 293.9 mm to (113.0, 135.0)
- moved C42 289.4 mm to (105.6, 130.0), turned to 270 degrees
- moved C1 287.4 mm to (108.6, 106.8), turned to 270 degrees
- moved L2 287.0 mm to (113.2, 129.8)
- moved C38 285.9 mm to (109.0, 137.4), turned to 180 degrees
- moved C41 285.0 mm to (109.2, 130.0), turned to 270 degrees
- moved C40 283.6 mm to (116.2, 134.2), turned to 90 degrees
- moved R12 280.6 mm to (116.8, 105.5), turned to 270 degrees
- moved U1 278.8 mm to (112.5, 107.5), turned to 180 degrees
- moved R14 277.8 mm to (116.8, 108.8), turned to 90 degrees
- moved R13 256.4 mm to (114.0, 104.8)
- moved C10 248.4 mm to (159.4, 126.8)
- moved C9 248.4 mm to (155.4, 129.5)
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Routing:
- net Net-(R35-Pad2): track 0.00 -> 2.16 mm
Other:
- board outline added: 116 x 107 mm

Commit message: placing components 85% done
Parts:
- added R18: 0.033, Resistor_SMD:R_2512_6332Metric, F.Cu at (195.4, 118.0)
- added R19: 0.068, Resistor_SMD:R_2512_6332Metric, F.Cu at (195.2, 130.6)
- moved R50 141.4 mm to (112.2, 72.6), turned to 180 degrees
- moved R53 140.5 mm to (121.8, 67.2)
- moved C47 133.0 mm to (127.4, 64.2), turned to 90 degrees
- moved U10 131.3 mm to (123.4, 64.2)
- moved R22 48.2 mm to (193.0, 82.2)
- moved X1 48.0 mm to (101.0, 128.4)
- moved R24 47.1 mm to (196.9, 77.8)
- moved R25 47.1 mm to (188.8, 77.0)
- moved R23 46.4 mm to (193.0, 76.4)
- moved C24 43.5 mm to (100.8, 131.0)
- moved R52 41.1 mm to (118.8, 66.2), turned to 270 degrees
- moved C10 36.1 mm to (190.0, 107.6)
- moved C9 36.1 mm to (186.0, 110.3)
- moved R15 36.1 mm to (178.5, 109.6)
- moved R54 35.2 mm to (119.2, 63.0), turned to 270 degrees
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Connections:
- Q8 pad 1: /BATT_VCC -> +BATT
- Q8 pad 2: /BATT_VCC -> +BATT
- Q8 pad 3: /BATT_VCC -> +BATT
- R50 pad 2: /BATT_VCC -> +BATT
- SW2 pad 1: /BATT_VCC -> +BATT

Commit message: new processor chip and add some suddenly missing footprints
Parts:
- C38: footprint Capacitor_SMD:C_0805_2012Metric -> Capacitor_SMD:C_0603_1608Metric
- C41, C42: footprint Capacitor_Tantalum_SMD:CP_EIA-3216-18_Kemet-A -> Capacitor_SMD:C_0603_1608Metric
- U5: value STM32G473CBU6-LQFP100 -> STM32G491MET6-LQFP80; footprint Package_QFP:LQFP-100_14x14mm_P0.5mm -> Package_QFP:LQFP-80_14x14mm_P0.65mm
- U8: value AMS1117-3.3 -> MCP1826S
- moved U8 51.4 mm to (126.0, 82.0)
Connections:
- net /MCU/PC5 renamed /MCU/A_PWM_15(PC5)
- net /MCU/QSPI1_BK2_IO0 renamed /MCU/QSPI1_BK2_IO0(ADC)
- net /MCU/QSPI1_BK2_IO1 renamed /MCU/QSPI1_BK2_IO1(ADC)
- net /MCU/QSPI1_BK2_IO2 renamed /MCU/QSPI1_BK2_IO2(ADC)
- net /MCU/QSPI1_BK2_IO3 renamed /MCU/QSPI1_BK2_IO3(ADC)
- net /MCU/SPI1_MISO renamed /MCU/SPI1_MISO(ADC)
- net /MCU/SPI1_MOSI renamed /MCU/SPI1_MOSI(ADC)
- net /MCU/SPI1_SCK renamed /MCU/SPI1_SCK(ADC)
- net /MCU/USART2_RX renamed /MCU/USART2_RX(ADC)
- net /MCU/USART2_TX renamed /MCU/USART2_TX(ADC)
- U5 pad 1: +3V3 -> Net-(U5-Pad1)
- U5 pad 28: +3V3 -> Net-(U5-Pad28)
- U5 pad 29: +3V3 -> Net-(U5-Pad29)
- U8 pad 1: GND -> +5V
- U8 pad 2: +3V3 -> GND
- U8 pad 3: +5V -> +3V3
