File: uHoubolt_PCB_PMU.sch (KiCad schematic (older format))
At the start: 14 parts, among them J1 Battery, J2 Umbilical, J3 Power, SW1 Power_1, SW2 Power_2, SW3 Pyro_1, SW4 Pyro_2

Commit message: Added ECU to PMU
Parts:
- removed F?: Polyfuse_Small, symbol Device:Polyfuse_Small
- removed H1, H2, H3, H4: M3, MountingHole:MountingHole_3.2mm_M3_Pad_Via, symbol Mechanical:MountingHole_Pad
- removed J1: Battery, Connector_PinSocket_2.54mm:PinSocket_1x02_P2.54mm_Vertical, symbol Connector_Generic:Conn_01x02
- removed J2: Umbilical, Connector_PinSocket_2.54mm:PinSocket_1x04_P2.54mm_Horizontal, symbol Connector_Generic:Conn_01x04
- removed J3: Power, TXV_Library_Footprints:Molex_MegaFit_1x03, symbol Connector_Generic:Conn_01x03
- removed Q?: Q_PMOS_GDS, symbol Device:Q_PMOS_GDS
- removed R?: R_Small, symbol Device:R_Small
- removed SW1: Power_1, TXV_Library_Footprints:D2F_A, symbol Switch:SW_Push_SPDT
- removed SW2: Power_2, TXV_Library_Footprints:D2F_A1, symbol Switch:SW_Push_SPDT
- removed SW3: Pyro_1, TXV_Library_Footprints:D2F_A, symbol Switch:SW_Push_SPDT
- removed SW4: Pyro_2, TXV_Library_Footprints:D2F_A1, symbol Switch:SW_Push_SPDT
Connections:
- no-connect marks 2 -> 0
Other:
- note removed: "Akkulader\n5V Buck\nSTM\n2x CAN\nBeeper\n2-4x 5V/Bat High Side switch"

Commit message: Revert "Added ECU to PMU"
This reverts commit 9e77d8288f64199274fc49822545c9b66851eb22.
Parts:
- added C1: 470n, Capacitor_SMD:C_0603_1608Metric, symbol Device:C
- added C10: 100n, Capacitor_SMD:C_0603_1608Metric, symbol Device:C_Small
- added C11: 100n, Capacitor_SMD:C_0402_1005Metric, symbol Device:C_Small
- added C12, C13: 2.2n, Capacitor_SMD:C_0603_1608Metric, symbol Device:C_Small
- added C14: 22u, Capacitor_SMD:C_0805_2012Metric, symbol Device:C_Small
- added C2, C3: 100n, Capacitor_SMD:C_0402_1005Metric, symbol Device:C
- added C4: 22u, Capacitor_SMD:C_0805_2012Metric, symbol Device:CP
- added C5: C, Capacitor_SMD:C_0603_1608Metric, symbol Device:C
- added C6: C, Capacitor_SMD:C_0805_2012Metric, symbol Device:C
- added C7: 10u, Capacitor_SMD:C_0805_2012Metric, symbol Device:C_Small
- added C8, C9: 4.7u, Capacitor_SMD:C_0603_1608Metric, symbol Device:C_Small
- added D1: 30V, Diode_SMD:D_SOD-123F, symbol Device:D_TVS
- added D2: 3.3V, Diode_SMD:D_SOD-323F, symbol Device:D_Zener
- added D3, D4: LED, LED_SMD:LED_0603_1608Metric, symbol Device:LED
- added D5: D_Schottky, Diode_SMD:D_0805_2012Metric_Castellated, symbol Device:D_Schottky
- added D6: D_Schottky_Small, Diode_SMD:D_0805_2012Metric_Castellated, symbol Device:D_Schottky_Small
- added H1, H2, H3, H4: M3, MountingHole:MountingHole_3.2mm_M3_Pad_Via, symbol Mechanical:MountingHole_Pad
- added J1: Umbilical, TXV_LIB:Molex_Nano-Fit_105309-xx02_1x02_P2.50mm_Vertical, symbol Connector_Generic:Conn_01x02
- added J2: Battery, TXV_LIB:Molex_Nano-Fit_105309-xx02_1x02_P2.50mm_Vertical, symbol Connector_Generic:Conn_01x02
- added J3: Power, TXV_Library_Footprints:Molex_MegaFit_1x03, symbol Connector_Generic:Conn_01x03
- added J4: Cam0, TXV_LIB:Molex_SL_1x2_Vertical, symbol Connector_Generic:Conn_01x02
- added J5: Batterycells, Connector_JST:JST_GH_BM04B-GHS-TBT_1x04-1MP_P1.25mm_Vertical, symbol Connector_Generic_MountingPin:Conn_01x04_MountingPin
- added J6: Cam1, TXV_LIB:Molex_SL_1x2_Vertical, symbol Connector_Generic:Conn_01x02
- added J7: Cam2, TXV_LIB:Molex_SL_1x2_Vertical, symbol Connector_Generic:Conn_01x02
- added L1, L2: L, TXV_Library_Footprints:SRN4018TA-4R7M, symbol Device:L
- added Q1, Q3, Q4: Q_PMOS_DGS, TXV_Library_Footprints:PG_TSDSON-8, symbol Device:Q_PMOS_DGS
- added Q2: BSZ0902NSATMA1, TXV_Library_Footprints:PG_TSDSON-8, symbol TXV_Library_Symbols:BSZ0902NSATMA1
- added R1, R15, R19, R23, R24, R25, R26, R27: R_Small, Resistor_SMD:R_0603_1608Metric, symbol Device:R_Small
- added R10, R2: 22k, Resistor_SMD:R_0603_1608Metric, symbol Device:R
- added R11: 2.7k, Resistor_SMD:R_0603_1608Metric, symbol Device:R
- added R14, R18: 200, Resistor_SMD:R_0603_1608Metric, symbol Device:R_Small
- added R20, R21, R22: R, Resistor_SMD:R_0603_1608Metric, symbol Device:R
- added R3: 1k1, Resistor_SMD:R_0603_1608Metric, symbol Device:R
- added R4: 2k4, Resistor_SMD:R_0603_1608Metric, symbol Device:R
- added R5: NP, Resistor_SMD:R_0603_1608Metric, symbol Device:R
- added R6: 2m, Resistor_SMD:R_1206_3216Metric, symbol Device:R
- added R7: 0R, Resistor_SMD:R_0603_1608Metric, symbol Device:R
- added R9: 47k, Resistor_SMD:R_0603_1608Metric, symbol Device:R
- added SW1: Power_1, TXV_Library_Footprints:D2F_A, symbol Switch:SW_Push_SPDT
- added SW2: Power_2, TXV_Library_Footprints:D2F_A1, symbol Switch:SW_Push_SPDT
- added SW3: Pyro_1, TXV_Library_Footprints:D2F_A, symbol Switch:SW_Push_SPDT
- added SW4: Pyro_2, TXV_Library_Footprints:D2F_A1, symbol Switch:SW_Push_SPDT
- added TH1: Thermistor_NTC, Connector_PinHeader_2.54mm:PinHeader_1x02_P2.54mm_Vertical, symbol Device:Thermistor_NTC
- added U1: LM5069, Package_SO:VSSOP-10_3x3mm_P0.5mm, symbol TXV_Library_Symbols:LM5069
- added U2: LMP8640 F, Package_TO_SOT_SMD:SOT-23-6, symbol TXV_Library_Symbols:INA180
- added U3: TS30041, Package_DFN_QFN:QFN-16-1EP_3x3mm_P0.5mm_EP1.75x1.75mm_ThermalVias, symbol TXV_Library_Symbols:TS30041
- added U4: MP26123, Package_DFN_QFN:QFN-16-1EP_4x4mm_P0.65mm_EP2.15x2.15mm_ThermalVias, symbol TXV_Library_Symbols:MP26123
- added U5: ECU, TXV_Library_Footprints:ECU_Footprint_simple, symbol TXV_Library_Symbols:ECU_simple
Connections:
- new net: Q1.2 (G), R1.2, SW1.2 (B), SW2.2 (B)
- new net: SW3.2 (B), SW4.1 (A)
- new net: D1.1 (A1), Q1.1 (D), R2.1, R5.1, R6.1, U1.2 (VIN), U2.3 (+)
- new net: C14.1, J2.2 (Pin_2), J5.1 (Pin_1), Q1.3 (S), R1.1, R27.1, U4.10 (BATT)
- new net: R2.2, R3.1, U1.3 (UVLO)
- new net: R3.2, R4.1, U1.4 (OVLO)
- new net: Q2.3 (D), R6.2, R7.2, U2.4 (-)
- new net: R5.2, R7.1, U1.1 (SENSE)
- new net: Q2.2 (G), U1.10 (GATE)
- new net: C1.1, U1.6 (TIMER)
- new net: R9.1, U1.7 (PWR)
- new net: C7.1, D5.2 (A), J1.2 (Pin_2), U4.1 (VCC)
- new net: L2.2, R27.2, U4.11 (CSP)
- new net: C10.1, U4.13 (TMR)
- new net: C11.2, U4.14 (BST)
- new net: C11.1, D6.1 (K), L2.1, U4.15 (SW)
- new net: C9.1, D5.1 (K), U4.16 (VIN)
- new net: C8.1, R22.1, R23.1, R24.1, U4.5 (VREF33), U4.7 (CELLS)
- new net: R26.2, U4.8 (COMPV)
- new net: R25.2, U4.9 (COMPI)
- new net: D3.2 (A), R23.2
- new net: C12.1, R26.1
- new net: C13.1, R25.1
- new net: D4.2 (A), R24.2
- new net: C5.1, L1.1, U3.1 (VSW), U3.12 (VSW), U3.13 (VSW), U3.16 (VSW)
- new net: C5.2, U3.10 (BST)
- new net: R20.1, R21.1, U3.5 (FB)
- new net: Q3.1 (D), U5.31 (+IN1)
- new net: Q3.2 (G), R14.1
- new net: R14.2, R15.2, R18.2, R19.2, U5.27 (+IN0)
- new net: Q4.1 (D), U5.35 (+IN2)
- new net: Q4.2 (G), R18.1
- new net +12V: C3.1, C4.1, J3.1 (Pin_1), Q2.1 (S), R10.1, SW3.1 (A), U1.9 (OUT), U3.11 (VCC), U3.2 (VCC), U3.3 (VCC), U5.17 (+12V)
- new net +5V: C6.2, J4.2 (Pin_2), J6.2 (Pin_2), J7.2 (Pin_2), L1.2, R20.2, U2.5 (V+), U5.19 (Pyro)
- new net Cell1: J5.3 (Pin_3), Q3.3 (S), R15.1
- new net Cell2: J5.2 (Pin_2), Q4.3 (S), R19.1
- new net GND: C1.2, C10.2, C12.2, C13.2, C14.2, C2.2, C3.2, C4.2, C6.1, C7.2, C8.2, C9.2, D1.2 (A2), D2.2 (A), D6.2 (A), H1.1, H2.1, H3.1, H4.1, J1.1 (Pin_1), J2.1 (Pin_1), J3.2 (Pin_2), J4.1 (Pin_1), J5.4 (Pin_4), J5.MP (MountPin), J6.1 (Pin_1), J7.1 (Pin_1), R11.2, R21.2, R4.2, R9.2, SW1.1 (A), SW2.1 (A), SW3.3 (C), SW4.3 (C), TH1.2, U1.5 (GND), U2.2 (GND), U3.14 (PGND), U3.15 (PGND), U3.17 (PAD), U3.4 (GND), U4.12 (GND), U4.6 (~EN), U5.0 (GND), U5.18 (GND), U5.29 (GND), U5.33 (GND), U5.37 (GND), U5.41 (GND), U5.45 (GND), U5.49 (GND)
- new net NTC: R22.2, TH1.1, U4.2 (NTC), U5.39 (+IN3)
- new net PYRO: J3.3 (Pin_3), SW4.2 (B)
- new net SUPPLY_CURRENT_SENSE: U2.1, U5.47 (+IN5)
- new net SUPPLY_VOLTAGE_SENSE: C2.1, D2.1 (K), R10.2, R11.1, U5.43 (+IN4)
- new net ~ACOK: D3.1 (K), U4.3 (~ACOK), U5.26 (+V0)
- new net ~CHGOK: D4.1 (K), U4.4 (~CHGOK), U5.30 (+V1)
- no-connect marks 0 -> 11
Other:
- note added: "Akkulader\n5V Buck\nSTM\n2x CAN\nBeeper\n2-4x 5V/Bat High Side switch"
- note added: "Over Current = \n2.03A = 55mV/27mOhm"
- note added: "Overvoltage 26.5V\n\n\nUndervoltage 18.3V"
- note added: "R1"
- note added: "R2"
- note added: "R3"
- note added: "Threshold = 2.5V\n\nUov / Uin = R3 / (R1 + R2 + R3)\nUuv / Uin = (R2 + R3) / (R1 + R2 + R3)\n"
