File: uHoubolt_PCB_PMU.sch (KiCad schematic (older format))
At the start: 69 parts, among them J1 Umbilical, J2 Battery, J3 Power, J4 Cam0, J5 Batterycells, J6 Cam1, J7 Cam2, Q1 Q_PMOS_DGS, Q2 BSZ0902NSATMA1, Q3 Q_PMOS_DGS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

Commit message: PMU ECU Combo (Fixed git mistakes)
Parts:
- added JP?: Jumper_3_Open, symbol Jumper:Jumper_3_Open
Connections:
- net +12V: now also JP?.3 (B); no longer U3.11 (VCC), U3.2 (VCC), U3.3 (VCC)
- net NTC: now also U5.30 (+V1); no longer U5.39 (+IN3)
- net PYRO: now also JP?.1 (A)
- net ~CHGOK: now also U5.39 (+IN3); no longer U5.30 (+V1)
- new net: U3.11 (VCC), U3.2 (VCC), U3.3 (VCC)
Other:
- note added: "TODO:\nAdd 5V Pad to connect ServoVoltage to 5V \n"
Changed lines of the file:
@@
 L power:+12V #PWR0104
 U 1 1 61D46601
-P 9125 7975
-F 0 "#PWR0104" H 9125 7825 50  0001 C CNN
-F 1 "+12V" H 9025 8125 50  0000 L CNN
-F 2 "" H 9125 7975 50  0001 C CNN
-F 3 "" H 9125 7975 50  0001 C CNN
-	1    9125 7975
+P 9500 7450
+F 0 "#PWR0104" H 9500 7300 50  0001 C CNN
+F 1 "+12V" H 9400 7600 50  0000 L CNN
+F 2 "" H 9500 7450 50  0001 C CNN
+F 3 "" H 9500 7450 50  0001 C CNN
+	1    9500 7450
 	1    0    0    -1
 $EndComp
@@
 	2925 2575 3325 2575
 Connection ~ 3325 2575
-Text Label 3725 6700 0    50   ~ 0
+Text Label 3725 7700 0    50   ~ 0
 ~CHGOK
 Text Label 3725 6250 0    50   ~ 0
@@
 Text Label 3800 3525 0    50   ~ 0
 NTC
-Text Label 3200 7700 0    50   ~ 0
+Text Label 3200 6700 0    50   ~ 0
 NTC
 Wire Wire Line
@@
 	2975 6375 2975 6800
 Wire Wire Line
-	3200 7700 4075 7700
+	3200 6700 4075 6700
 Connection ~ 3550 6350
 Wire Wire Line
@@
 	4075 6250 3725 6250
 Wire Wire Line
-	4075 6700 3725 6700
+	4075 7700 3725 7700
 NoConn ~ 10425 8925
 Wire Wire Line
@@
 	11725 5500 11725 5625
 NoConn ~ 9225 8475
+$Comp
+L Jumper:Jumper_3_Open JP?
+U 1 1 61C433FF
+P 9125 7575
+F 0 "JP?" H 9125 7799 50  0000 C CNN
+F 1 "Jumper_3_Open" H 9125 7708 50  0000 C CNN
+F 2 "" H 9125 7575 50  0001 C CNN
+F 3 "~" H 9125 7575 50  0001 C CNN
+	1    9125 7575
+	1    0    0    -1
+$EndComp
+$Comp
+L TXV_Library_Symbols:Pyro #PWR?
+U 1 1 61C662AA
+P 8750 7450
+F 0 "#PWR?" H 8750 7300 50  0001 C CNN
+F 1 "Pyro" H 8750 7600 50  0000 C CNN
+F 2 "" H 8750 7450 50  0001 C CNN
+F 3 "" H 8750 7450 50  0001 C CNN
+	1    8750 7450
+	1    0    0    -1
+$EndComp
+Wire Wire Line
+	9500 7575 9375 7575
+Wire Wire Line
+	8875 7575 8750 7575
+Wire Wire Line
+	8750 7575 8750 7450
+Wire Wire Line
+	9500 7450 9500 7575
+Wire Wire Line
+	9125 7950 9125 7725
+Text Notes 8025 5450 0    50   ~ 0
+TODO:\nAdd 5V Pad to connect ServoVoltage to 5V \n
 $EndSCHEMATC

Commit message: PMU Layout
Parts:
- added C15, C17: 22u, Capacitor_SMD:C_0805_2012Metric, symbol Device:C
- added C16, C19: 100n, Capacitor_SMD:C_0402_1005Metric, symbol Device:C
- added C18: 22u, Capacitor_SMD:C_0805_2012Metric, symbol Device:C_Small
- added G?: SpaceTeam_LOGO, symbol TXV_Library_Symbols:SpaceTeam_LOGO
- added JP2: Jumper_2_Open, Jumper:SolderJumper-2_P1.3mm_Open_RoundedPad1.0x1.5mm, symbol Device:Jumper_NO_Small
- C5: value C -> 100n; footprint Capacitor_SMD:C_0603_1608Metric -> Capacitor_SMD:C_0402_1005Metric
- C6: value C -> 22u
- C7: value 10u -> 22u
- D5: value D_Schottky -> PMEG3050EP; footprint Diode_SMD:D_0805_2012Metric_Castellated -> Diode_SMD:D_SOD-128
- D6: value D_Schottky_Small -> PMEG3050EP; footprint Diode_SMD:D_0805_2012Metric_Castellated -> Diode_SMD:D_SOD-128
- J1, J2: footprint TXV_LIB:Molex_Nano-Fit_105309-xx02_1x02_P2.50mm_Vertical -> TXV_Library_Footprints:Molex_Nano-Fit_105309-xx02_1x02_P2.50mm_Vertical
- J3: footprint TXV_Library_Footprints:Molex_MegaFit_1x03 -> TXV_Library_Footprints:Molex_MegaFit_1x03_Vertical
- J4, J6, J7: footprint TXV_LIB:Molex_SL_1x2_Vertical -> TXV_Library_Footprints:Molex_SL_1x2_Vertical
- JP1: renamed from JP?; footprint (none) -> TXV_Library_Footprints:Jumper3_6x2mm
- L1, L2: value L -> 4.7u
- R1, R15, R19: value R_Small -> 10k
- R10, R2: value 22k -> R
- R11: value 2.7k -> R
- R22: value R -> 10k
- R23, R24: value R_Small -> 120
- R25: value R_Small -> 750
- R26: value R_Small -> 2.5k
- R27: value R_Small -> 140m; footprint Resistor_SMD:R_0603_1608Metric -> Resistor_SMD:R_0805_2012Metric
- R3: value 1k1 -> R
- R4: value 2k4 -> R
Connections:
- net +5V: now also C17.2, C19.1
- net GND: now also J1.2 (Pin_2), J2.2 (Pin_2), C15.1, C16.2, C17.1, C18.2, C19.2, JP2.2; no longer J1.1 (Pin_1), J2.1 (Pin_1)
- net Vin: now reaches D1.1 (A1), Q1.1 (D), R2.1, R5.1, R6.1, U1.2 (VIN), U2.3 (+)
- net Vbat: now reaches C14.1, Q1.3 (S), R1.1, R27.1, U4.10 (BATT)
- net Vbat: now also J2.1 (Pin_1), C18.1; no longer J2.2 (Pin_2), J5.1 (Pin_1)
- net Vcharge: now reaches C7.1, D5.2 (A), U4.1 (VCC)
- net Vcharge: now also J1.1 (Pin_1); no longer J1.2 (Pin_2)
- net +3V3: now reaches C8.1, R22.1, R23.1, R24.1, U4.5 (VREF33)
- net +3V3: no longer U4.7 (CELLS)
- net at JP1.2 (C): now also U3.11 (VCC), U3.2 (VCC), U3.3 (VCC), C15.2, C16.1
- new net: JP2.1, U4.7 (CELLS)
- no-connect marks 11 -> 16
Other:
- note added: "I_charge = 200mV / RS1 \nRS1 = 200mV / I_charge"
- note removed: "TODO:\nAdd 5V Pad to connect ServoVoltage to 5V \n"
- moved on the sheet: J2, R22

Commit message: New Layout
Parts:
- G1: renamed from G?; footprint (none) -> TXV_Library_Footprints:ST_Logo_new
Changed lines of the file:
@@
 Connection ~ 11500 1475
 $Comp
-L TXV_Library_Symbols:SpaceTeam_LOGO G?
+L TXV_Library_Symbols:SpaceTeam_LOGO G1
 U 1 1 6259FDE3
 P 8900 1775
-F 0 "G?" H 8900 1569 60  0001 C CNN
+F 0 "G1" H 8900 1569 60  0001 C CNN
 F 1 "SpaceTeam_LOGO" H 8900 1981 60  0001 C CNN
-F 2 "" H 8900 1775 50  0001 C CNN
+F 2 "TXV_Library_Footprints:ST_Logo_new" H 8900 1775 50  0001 C CNN
 F 3 "" H 8900 1775 50  0001 C CNN
 	1    8900 1775

Commit message: Release Version of PMU V1
Parts:
- removed C2: 100n, Capacitor_SMD:C_0402_1005Metric, symbol Device:C
- removed D2: 3.3V, Diode_SMD:D_SOD-323F, symbol Device:D_Zener
- removed R10, R11: R, Resistor_SMD:R_0603_1608Metric, symbol Device:R
- added J8: 12V, TXV_Library_Footprints:Molex_SL_1x2_Vertical, symbol Connector_Generic:Conn_01x02
- added Q5, Q6: BC817W, Package_TO_SOT_SMD:SOT-323_SC-70, symbol Transistor_BJT:BC817W
- added R12, R8: 10k, Resistor_SMD:R_0603_1608Metric, symbol Device:R_Small
- Q1, Q3, Q4: value Q_PMOS_DGS -> BSZ0905PNSATMA1; symbol Device:Q_PMOS_DGS -> Device:Q_PMOS_SGD
Connections:
- net SUPPLY_VOLTAGE_SENSE is gone; now on net ~ACOK: U5.43 (+IN4)
- net +12V: now also J8.1 (Pin_1)
- net +5V: now also J4.1 (Pin_1), J6.1 (Pin_1), J7.1 (Pin_1); no longer J4.2 (Pin_2), J6.2 (Pin_2), J7.2 (Pin_2)
- net Cell1: now also Q3.1 (S); no longer Q3.3 (S)
- net Cell2: now also Q4.1 (S); no longer Q4.3 (S)
- net GND: now also J4.2 (Pin_2), J6.2 (Pin_2), J7.2 (Pin_2), J8.2 (Pin_2), Q5.2 (E), Q6.2 (E); no longer J4.1 (Pin_1), J6.1 (Pin_1), J7.1 (Pin_1)
- net Vbat: now also Q1.1 (S); no longer Q1.3 (S)
- net Vin: now also Q1.3 (D); no longer Q1.1 (D)
- net ~ACOK: no longer U5.26 (+V0)
- net at U5.31 (+IN1): now also Q3.3 (D); no longer Q3.1 (D)
- net at U5.35 (+IN2): now also Q4.3 (D); no longer Q4.1 (D)
- new net: Q5.3 (C), R14.2, R15.2
- new net: Q6.3 (C), R18.2, R19.2
- new net: Q5.1 (B), R8.1
- new net: R12.2, R8.2, U5.27 (+IN0)
- new net: Q6.1 (B), R12.1
- no-connect marks 16 -> 17
Other:
- moved on the sheet: Q3, Q4, R14, R15, R18, R19
