File: uHoubolt_PCB_PMU.kicad_pcb (KiCad board)
At the start: 2 copper layers, 117.8 x 90 mm, 11 parts, among them J1 Conn_01x02, J2 Conn_01x04, J3 Conn_01x03, SW1 Power_1, SW2 Power_2, SW3 Pyro_1, SW4 Pyro_2

Commit message: PMU Layout
Parts:
- added C1: 470n, Capacitor_SMD:C_0603_1608Metric, F.Cu at (174.8, 125.2)
- added C10: 100n, Capacitor_SMD:C_0603_1608Metric, F.Cu at (155.8, 131.4)
- added C11: 100n, Capacitor_SMD:C_0402_1005Metric, F.Cu at (151.6, 130.1)
- added C12: 2.2n, Capacitor_SMD:C_0603_1608Metric, F.Cu at (156.4, 136.8)
- added C13: 2.2n, Capacitor_SMD:C_0603_1608Metric, F.Cu at (156.4, 133.6)
- added C14: 22u, Capacitor_SMD:C_0805_2012Metric, F.Cu at (161.4, 129.0)
- added C15: 22u, Capacitor_SMD:C_0805_2012Metric, F.Cu at (151.0, 69.0)
- added C16: 100n, Capacitor_SMD:C_0402_1005Metric, F.Cu at (150.8, 67.0)
- added C17: 22u, Capacitor_SMD:C_0805_2012Metric, F.Cu at (147.6, 69.0)
- added C18: 22u, Capacitor_SMD:C_0805_2012Metric, F.Cu at (163.4, 129.0)
- added C19: 100n, Capacitor_SMD:C_0402_1005Metric, F.Cu at (168.8, 115.6)
- added C2: 100n, Capacitor_SMD:C_0402_1005Metric, F.Cu at (102.0, 114.8)
- added C3: 100n, Capacitor_SMD:C_0402_1005Metric, F.Cu at (173.4, 119.7)
- added C4: 22u, Capacitor_SMD:C_0805_2012Metric, F.Cu at (175.0, 119.3)
- added C5: 100n, Capacitor_SMD:C_0402_1005Metric, F.Cu at (152.7, 60.6)
- added C6: 22u, Capacitor_SMD:C_0805_2012Metric, F.Cu at (147.6, 67.0)
- added C7: 22u, Capacitor_SMD:C_0805_2012Metric, F.Cu at (142.0, 129.2)
- added C8: 4.7u, Capacitor_SMD:C_0603_1608Metric, F.Cu at (150.0, 136.8)
- added C9: 4.7u, Capacitor_SMD:C_0603_1608Metric, F.Cu at (148.0, 129.0)
- added D1: 30V, Diode_SMD:D_SOD-123F, F.Cu at (162.6, 119.8)
- added D2: 3.3V, Diode_SMD:D_SOD-323F, F.Cu at (101.8, 118.2)
- added D3: LED, LED_SMD:LED_0603_1608Metric, F.Cu at (145.8, 136.2)
- added D4: LED, LED_SMD:LED_0603_1608Metric, F.Cu at (147.4, 136.2)
- added D5: PMEG3050EP, Diode_SMD:D_SOD-128, F.Cu at (145.4, 129.4)
- added D6: PMEG3050EP, Diode_SMD:D_SOD-128, F.Cu at (156.8, 128.6)
- added G1: SpaceTeam_LOGO, TXV_Library_Footprints:ST_Logo_new, F.Cu at (168.5, 75.0)
- added J4: Cam0, TXV_Library_Footprints:Molex_SL_1x2_Vertical, F.Cu at (118.0, 62.0)
- added J5: Batterycells, Connector_JST:JST_GH_BM04B-GHS-TBT_1x04-1MP_P1.25mm_Vertical, F.Cu at (181.0, 128.2)
- added J6: Cam1, TXV_Library_Footprints:Molex_SL_1x2_Vertical, F.Cu at (125.0, 62.0)
- added J7: Cam2, TXV_Library_Footprints:Molex_SL_1x2_Vertical, F.Cu at (132.0, 62.0)
- added JP1: Jumper_3_Open, TXV_Library_Footprints:Jumper3_6x2mm, B.Cu at (190.8, 81.8)
- added JP2: Jumper_2_Open, Jumper:SolderJumper-2_P1.3mm_Open_RoundedPad1.0x1.5mm, F.Cu at (151.7, 139.2)
- added L1: 4.7u, TXV_Library_Footprints:SRN4018TA-4R7M, F.Cu at (148.4, 63.7)
- added L2: 4.7u, TXV_Library_Footprints:SRN4018TA-4R7M, F.Cu at (151.4, 127.4)
- added Q1: Q_PMOS_DGS, TXV_Library_Footprints:PG_TSDSON-8, F.Cu at (159.4, 124.0)
- added Q2: BSZ0902NSATMA1, TXV_Library_Footprints:PG_TSDSON-8, F.Cu at (170.8, 120.8)
- added Q3: Q_PMOS_DGS, TXV_Library_Footprints:PG_TSDSON-8, F.Cu at (183.4, 136.0)
- added Q4: Q_PMOS_DGS, TXV_Library_Footprints:PG_TSDSON-8, F.Cu at (179.0, 136.0)
- added R1: 10k, Resistor_SMD:R_0603_1608Metric, F.Cu at (157.2, 123.0)
- added R10: R, Resistor_SMD:R_0603_1608Metric, F.Cu at (101.5, 120.0)
- added R11: R, Resistor_SMD:R_0603_1608Metric, F.Cu at (101.5, 116.2)
- added R14: 200, Resistor_SMD:R_0603_1608Metric, F.Cu at (183.8, 133.8)
- added R15: 10k, Resistor_SMD:R_0603_1608Metric, F.Cu at (183.8, 132.2)
- added R18: 200, Resistor_SMD:R_0603_1608Metric, F.Cu at (179.5, 133.8)
- added R19: 10k, Resistor_SMD:R_0603_1608Metric, F.Cu at (179.5, 132.2)
- added R2: R, Resistor_SMD:R_0603_1608Metric, F.Cu at (161.6, 123.8)
- added R20: R, Resistor_SMD:R_0603_1608Metric, F.Cu at (155.9, 63.0)
- added R21: R, Resistor_SMD:R_0603_1608Metric, F.Cu at (155.9, 66.1)
- added R22: 10k, Resistor_SMD:R_0603_1608Metric, F.Cu at (144.2, 139.2)
- added R23: 120, Resistor_SMD:R_0603_1608Metric, F.Cu at (145.8, 139.2)
- added R24: 120, Resistor_SMD:R_0603_1608Metric, F.Cu at (147.4, 139.2)
- added R25: 750, Resistor_SMD:R_0603_1608Metric, F.Cu at (156.4, 135.2)
- added R26: 2.5k, Resistor_SMD:R_0603_1608Metric, F.Cu at (153.2, 136.8)
- added R27: 140m, Resistor_SMD:R_0805_2012Metric, F.Cu at (155.4, 126.0)
- added R3: R, Resistor_SMD:R_0603_1608Metric, F.Cu at (163.2, 125.8)
- added R4: R, Resistor_SMD:R_0603_1608Metric, F.Cu at (164.7, 125.8)
- added R5: NP, Resistor_SMD:R_0603_1608Metric, F.Cu at (164.7, 122.0)
- added R6: 2m, Resistor_SMD:R_1206_3216Metric, F.Cu at (166.2, 119.2)
- added R7: 0R, Resistor_SMD:R_0603_1608Metric, F.Cu at (167.0, 121.2)
- added R9: 47k, Resistor_SMD:R_0603_1608Metric, F.Cu at (174.8, 123.8)
- added TH1: Thermistor_NTC, Connector_PinHeader_2.54mm:PinHeader_1x02_P2.54mm_Vertical, F.Cu at (174.4, 130.6)
- added U1: LM5069, Package_SO:VSSOP-10_3x3mm_P0.5mm, F.Cu at (168.8, 124.0)
- added U2: LMP8640 F, Package_TO_SOT_SMD:SOT-23-6, F.Cu at (166.2, 116.1)
- added U3: TS30041, Package_DFN_QFN:QFN-16-1EP_3x3mm_P0.5mm_EP1.75x1.75mm_ThermalVias, F.Cu at (152.9, 63.6)
- added U4: MP26123, Package_DFN_QFN:QFN-16-1EP_4x4mm_P0.65mm_EP2.15x2.15mm_ThermalVias, F.Cu at (151.6, 133.3)
- added U5: ECU, TXV_Library_Footprints:ECU_Footprint_simple, F.Cu at (120.0, 101.0)
- H1, H2, H3, H4: value MountingHole_Pad -> M3
- J1: value Conn_01x02 -> Umbilical; footprint Connector_PinSocket_2.54mm:PinSocket_1x02_P2.54mm_Vertical -> TXV_Library_Footprints:Molex_Nano-Fit_105309-xx02_1x02_P2.50mm_Vertical; moved to B.Cu
- J2: value Conn_01x04 -> Battery; footprint Connector_PinSocket_2.54mm:PinSocket_1x04_P2.54mm_Horizontal -> TXV_Library_Footprints:Molex_Nano-Fit_105309-xx02_1x02_P2.50mm_Vertical
- J3: value Conn_01x03 -> Power; footprint TXV_Library_Footprints:Molex_MegaFit_1x03 -> TXV_Library_Footprints:Molex_MegaFit_1x03_Vertical; moved to B.Cu
- moved J2 83.3 mm to (167.8, 128.5), turned to 90 degrees
- moved J1 70.9 mm to (142.3, 132.2), turned to 180 degrees
- moved J3 11.7 mm to (159.5, 53.0), turned to 180 degrees
- moved H1 5.11 mm to (109.0, 62.0)
- moved H2 5.11 mm to (171.0, 62.0)
- moved H3 5.11 mm to (109.0, 138.0)
- moved H4 5.11 mm to (171.0, 138.0)
Connections:
- H1 pad 1: Net-(H1-Pad1) -> GND
- H2 pad 1: Net-(H2-Pad1) -> GND
- H3 pad 1: Net-(H3-Pad1) -> GND
- H4 pad 1: Net-(H4-Pad1) -> GND
- J1 pad 1: Net-(J1-Pad1) -> /Vcharge
- J1 pad 2: Net-(J1-Pad2) -> GND
- J2 pad 1: Net-(J2-Pad1) -> /Vbat
- J2 pad 2: Net-(J2-Pad2) -> GND
- J3 pad 1: Net-(J3-Pad1) -> +12V
- J3 pad 2: Net-(J3-Pad2) -> GND
- J3 pad 3: Net-(J3-Pad3) -> PYRO
- SW1 pad 1: Net-(SW1-Pad1) -> GND
- SW1 pad 2: Net-(SW1-Pad2) -> Net-(Q1-Pad2)
- SW1 pad 3: Net-(SW1-Pad3) -> (no net)
- SW2 pad 1: Net-(SW2-Pad1) -> GND
- SW2 pad 2: Net-(SW2-Pad2) -> Net-(Q1-Pad2)
- SW2 pad 3: Net-(SW2-Pad3) -> (no net)
- SW3 pad 1: Net-(SW3-Pad1) -> +12V
- SW3 pad 3: Net-(SW3-Pad3) -> GND
- SW4 pad 1: Net-(SW4-Pad1) -> Net-(SW3-Pad2)
- SW4 pad 2: Net-(SW4-Pad2) -> PYRO
- SW4 pad 3: Net-(SW4-Pad3) -> GND
Routing:
- net +12V: track 0.00 -> 225.1 mm, vias 0 -> 15
- net +5V: track 0.00 -> 146.2 mm
- net Net-(Q3-Pad1): track 0.00 -> 100.1 mm, vias 0 -> 2
- net Net-(Q4-Pad1): track 0.00 -> 99.8 mm, vias 0 -> 2
- net Net-(R14-Pad2): track 0.00 -> 89.4 mm, vias 0 -> 3
- net /SUPPLY_CURRENT_SENSE: track 0.00 -> 88.7 mm, vias 0 -> 2
- net /NTC: track 0.00 -> 86.7 mm, vias 0 -> 3
- net PYRO: track 0.00 -> 75.0 mm
- net Net-(Q1-Pad2): track 0.00 -> 58.5 mm, vias 0 -> 1
- net /~CHGOK: track 0.00 -> 53.5 mm
- net Net-(C15-Pad2): track 0.00 -> 53.4 mm, vias 0 -> 8
- net /~ACOK: track 0.00 -> 47.0 mm
- net GND: track 0.00 -> 37.6 mm, vias 0 -> 1
- net Net-(SW3-Pad2): track 0.00 -> 30.5 mm
- net /Vbat: track 0.00 -> 27.6 mm, vias 0 -> 2
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- added copper zone on B.Cu, net +12V
- added copper zone on F.Cu, net +12V
- added copper zone on F.Cu, net +5V
- added copper zone on F.Cu, net /Vbat
- added copper zone on F.Cu, net /Vcharge
- added copper zone on F.Cu, net /Vin
- added copper zone on B.Cu, net GND
- added copper zone on F.Cu, net GND
- added copper zone on F.Cu, net Net-(C11-Pad1)
- added copper zone on B.Cu, net Net-(C15-Pad2)
- added copper zone on F.Cu, net Net-(C15-Pad2)
- added copper zone on F.Cu, net Net-(C5-Pad1)
- added copper zone on F.Cu, net Net-(L2-Pad2)
Other:
- board size 117.8 x 90 mm -> 118.8 x 98 mm
- rule via_min_size: 0.4 -> 0.3
- board text added: "PMU v1.0 SN:"
- board text removed: "Leinenseite"
- board text removed: "Schaltbare Ausgänge"

Commit message: New Layout
Parts:
- J4, J6, J7: moved to B.Cu
- moved R22 93.8 mm to (116.0, 49.7), turned to 0 degrees
- moved R23 93.4 mm to (114.5, 51.2), turned to 0 degrees
- moved R24 92.4 mm to (114.5, 52.8), turned to 0 degrees
- moved JP2 89.7 mm to (115.8, 57.0), turned to 90 degrees
- moved D3 89.6 mm to (117.5, 51.2), turned to 180 degrees
- moved D4 88.6 mm to (117.5, 52.8), turned to 180 degrees
- moved C8 87.5 mm to (118.2, 55.3), turned to 270 degrees
- moved J1 86.3 mm to (123.2, 48.0), turned to 90 degrees
- moved R26 85.8 mm to (118.2, 58.5), turned to 90 degrees
- moved C12 83.8 mm to (118.2, 62.2), turned to 270 degrees
- moved C7 83.1 mm to (126.5, 47.6), turned to 90 degrees
- moved U4 82.0 mm to (121.7, 56.9), turned to 270 degrees
- moved R25 81.7 mm to (119.8, 62.2), turned to 90 degrees
- moved D5 80.6 mm to (126.6, 51.0), turned to 180 degrees
- moved C13 79.5 mm to (121.4, 62.2), turned to 270 degrees
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Routing:
- net /Cell1: track 9.40 -> 109.3 mm
- net /Cell2: track 9.85 -> 107.0 mm
- net /NTC: track 86.7 -> 177.3 mm, vias 3 -> 2
- net +5V: track 146.2 -> 85.8 mm
- net /~ACOK: track 47.0 -> 103.9 mm, vias 0 -> 2
- net +12V: track 225.1 -> 174.0 mm, vias 15 -> 7
- net /SUPPLY_CURRENT_SENSE: track 88.7 -> 136.7 mm
- net Net-(Q3-Pad1): track 100.1 -> 53.3 mm, vias 2 -> 0
- net /~CHGOK: track 53.5 -> 94.7 mm, vias 0 -> 2
- net Net-(C15-Pad2): track 53.4 -> 14.2 mm, vias 8 -> 7
- net Net-(Q4-Pad1): track 99.8 -> 60.8 mm, vias 2 -> 0
- net Net-(R14-Pad2): track 89.4 -> 60.8 mm, vias 3 -> 2
- net /Vbat: track 27.6 -> 9.90 mm
- net PYRO: track 75.0 -> 87.5 mm
- net Net-(Q2-Pad3): track 10.7 -> 0.00 mm
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- added copper zone on F.Cu, net Net-(Q1-Pad2)
- added copper zone on F.Cu, net Net-(Q2-Pad3)
- removed copper zone on F.Cu, net /Vcharge
Other:
- board size 118.8 x 98 mm -> 118.5 x 100 mm
- board text removed: "Akkumanagement"

Commit message: Release Version of PMU V1
Parts:
- removed C2: 100n, Capacitor_SMD:C_0402_1005Metric
- removed D2: 3.3V, Diode_SMD:D_SOD-323F
- removed R10, R11: R, Resistor_SMD:R_0603_1608Metric
- added J8: 12V, TXV_Library_Footprints:Molex_SL_1x2_Vertical, B.Cu at (125.5, 50.0)
- added Q5: BC817W, Package_TO_SOT_SMD:SOT-323_SC-70, F.Cu at (146.0, 138.2)
- added Q6: BC817W, Package_TO_SOT_SMD:SOT-323_SC-70, F.Cu at (146.2, 132.0)
- added R12: 10k, Resistor_SMD:R_0603_1608Metric, F.Cu at (143.4, 132.0)
- added R8: 10k, Resistor_SMD:R_0603_1608Metric, F.Cu at (143.4, 136.6)
- Q1, Q3, Q4: value Q_PMOS_DGS -> BSZ0905PNSATMA1
- moved C7 12.1 mm to (115.7, 53.1), turned to 180 degrees
- moved R22 7.29 mm to (110.9, 54.9), turned to 180 degrees
- moved R1 6.50 mm to (172.6, 75.2)
- moved D5 5.98 mm to (121.9, 54.7)
- moved R18 5.88 mm to (150.0, 131.0), turned to 0 degrees
- moved R19 5.52 mm to (152.5, 131.8), turned to 90 degrees
- moved Q4 4.44 mm to (150.0, 133.8), turned to 270 degrees
- moved R14 4.21 mm to (150.0, 137.5), turned to 0 degrees
- moved J1 4.13 mm to (119.8, 50.4), turned to 0 degrees
- moved R15 4.03 mm to (152.5, 138.2), turned to 90 degrees
- moved R26 3.96 mm to (117.1, 62.3), turned to 0 degrees
- moved Q3 3.79 mm to (150.0, 140.2), turned to 270 degrees
- moved D4 3.74 mm to (117.0, 56.5)
- moved R24 3.74 mm to (114.0, 56.5)
- moved D3 3.74 mm to (117.0, 54.9)
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Connections:
- J4 pad 1: GND -> +5V
- J4 pad 2: +5V -> GND
- J6 pad 1: GND -> +5V
- J6 pad 2: +5V -> GND
- J7 pad 1: GND -> +5V
- J7 pad 2: +5V -> GND
- Q1 pad 1: /Vin -> /Vbat
- Q1 pad 3: /Vbat -> /Vin
- Q3 pad 1: Net-(Q3-Pad1) -> /Cell1
- Q3 pad 3: /Cell1 -> Net-(Q3-Pad3)
- Q4 pad 1: Net-(Q4-Pad1) -> /Cell2
- Q4 pad 3: /Cell2 -> Net-(Q4-Pad3)
- R14 pad 2: Net-(R14-Pad2) -> Net-(Q5-Pad3)
- R15 pad 2: Net-(R14-Pad2) -> Net-(Q5-Pad3)
- R18 pad 2: Net-(R14-Pad2) -> Net-(Q6-Pad3)
- R19 pad 2: Net-(R14-Pad2) -> Net-(Q6-Pad3)
- U5 pad 26: /~ACOK -> (no net)
- U5 pad 27: Net-(R14-Pad2) -> Net-(R12-Pad2)
- U5 pad 31: Net-(Q3-Pad1) -> Net-(Q3-Pad3)
- U5 pad 35: Net-(Q4-Pad1) -> Net-(Q4-Pad3)
- U5 pad 43: /SUPPLY_VOLTAGE_SENSE -> /~ACOK
Routing:
- net Net-(Q4-Pad3): track 0.00 -> 80.6 mm
- net Net-(Q3-Pad3): track 0.00 -> 71.6 mm
- net Net-(R14-Pad2): track 60.8 -> 0.00 mm, vias 2 -> 0
- net Net-(Q4-Pad1): track 60.8 -> 0.00 mm
- net Net-(Q3-Pad1): track 53.3 -> 0.00 mm
- net Net-(R12-Pad2): track 0.00 -> 47.6 mm
- net +12V: track 174.0 -> 135.2 mm
- net /SUPPLY_VOLTAGE_SENSE: track 16.2 -> 0.00 mm
- net /~ACOK: track 103.9 -> 90.1 mm
- net /Cell1: track 109.3 -> 98.1 mm
- net /Cell2: track 107.0 -> 97.8 mm
- net /NTC: track 177.3 -> 168.5 mm, vias 2 -> 3
- net +5V: track 85.8 -> 93.2 mm
- net Net-(Q5-Pad3): track 0.00 -> 7.18 mm
- net Net-(Q6-Pad3): track 0.00 -> 7.00 mm
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- added copper zone on F.Cu, net /Vcharge
- removed copper zone on F.Cu, net Net-(Q1-Pad2)
Other:
- board text added: "+"
- board text added: "12V"
- board text added: "BALANCE"
- board text added: "BATT"
- board text added: "Charger"
- board text added: "ECU"
- board text added: "GND"
- board text added: "JLCJLCJLCJLC"
- board text added: "PMU v1.0"
- board text added: "PYRO"
- board text added: "Temp"
- board text removed: "PMU v1.0 SN:"

Commit message: WIP PMU V2
Parts:
- removed J4: Cam0, TXV_Library_Footprints:Molex_SL_1x2_Vertical
- removed J6: Cam1, TXV_Library_Footprints:Molex_SL_1x2_Vertical
- removed J7: Cam2, TXV_Library_Footprints:Molex_SL_1x2_Vertical
- removed JP1: Jumper_3_Open, TXV_Library_Footprints:Jumper3_6x2mm
- added C2: 100n, Capacitor_SMD:C_0603_1608Metric, F.Cu at (178.4, 63.1)
- added C20: 100n, Capacitor_SMD:C_0603_1608Metric, F.Cu at (175.7, 64.0)
- added C21: 100n, Capacitor_SMD:C_0603_1608Metric, F.Cu at (173.5, 72.3)
- added C22: 2u2, Capacitor_SMD:C_0603_1608Metric, F.Cu at (157.1, 64.3)
- added C23: 100n, Capacitor_SMD:C_0603_1608Metric, F.Cu at (176.0, 61.0)
- added C24: 2u2, Capacitor_SMD:C_0603_1608Metric, F.Cu at (158.5, 60.0)
- added C25: 100n, Capacitor_SMD:C_0603_1608Metric, F.Cu at (170.1, 54.1)
- added C26: 100n, Capacitor_SMD:C_0603_1608Metric, F.Cu at (167.8, 54.9)
- added C27: 100n, Capacitor_SMD:C_0603_1608Metric, F.Cu at (154.1, 54.5)
- added C28: 100n, Capacitor_SMD:C_0603_1608Metric, F.Cu at (161.9, 73.0)
- added C29: 100n, Capacitor_SMD:C_0603_1608Metric, F.Cu at (176.5, 69.8)
- added C30: 100n, Capacitor_SMD:C_0603_1608Metric, F.Cu at (158.7, 64.3)
- added C31: 2u2, Capacitor_SMD:C_0603_1608Metric, F.Cu at (360.9, 250.9)
- added C32: 100n, Capacitor_SMD:C_0402_1005Metric, F.Cu at (117.3, 57.3)
- added C33: 100n, Capacitor_SMD:C_0402_1005Metric, F.Cu at (117.3, 67.3)
- added C34: 2u2, Capacitor_SMD:C_0603_1608Metric, F.Cu at (171.0, 76.0)
- added C35: 100n, Capacitor_SMD:C_0603_1608Metric, F.Cu at (169.5, 76.0)
- added C36: 2u2, Capacitor_SMD:C_0603_1608Metric, F.Cu at (356.7, 251.4)
- added C37: 100n, Capacitor_SMD:C_0402_1005Metric, F.Cu at (121.3, 59.8)
- added C38: 100n, Capacitor_SMD:C_0402_1005Metric, F.Cu at (121.3, 69.8)
- added C39: 10n, Capacitor_SMD:C_0603_1608Metric, F.Cu at (168.0, 76.0)
- added C40: 100n, Capacitor_SMD:C_0603_1608Metric, F.Cu at (166.5, 78.8)
- added C41: 100n, Capacitor_SMD:C_0603_1608Metric, F.Cu at (175.3, 54.9)
- added C42: 100n, Capacitor_SMD:C_0603_1608Metric, F.Cu at (177.7, 57.2)
- added C43: 22u, Capacitor_SMD:C_0805_2012Metric, F.Cu at (170.7, 120.0)
- added C44: 22u, Capacitor_SMD:C_0805_2012Metric, F.Cu at (97.0, 77.8)
- added C45: 100n, Capacitor_SMD:C_0402_1005Metric, F.Cu at (95.0, 77.6)
- added C46: 100n, Capacitor_SMD:C_0402_1005Metric, F.Cu at (89.0, 77.0)
- added C47: 22u, Capacitor_SMD:C_0805_2012Metric, F.Cu at (97.0, 81.2)
- added C48: 22u, Capacitor_SMD:C_0805_2012Metric, F.Cu at (95.0, 81.2)
- added D10: OUT 1, LED_SMD:LED_0603_1608Metric, F.Cu at (90.0, 97.1)
- added D11: OUT 1, LED_SMD:LED_0603_1608Metric, F.Cu at (98.3, 97.1)
- added D12: OUT 1, LED_SMD:LED_0603_1608Metric, F.Cu at (106.8, 97.1)
- added D13: Shottky, Diode_SMD:D_SOD-123F, F.Cu at (93.0, 92.2)
- added D14: Shottky, Diode_SMD:D_SOD-123F, F.Cu at (101.5, 92.2)
- added D15: Shottky, Diode_SMD:D_SOD-123F, F.Cu at (109.8, 92.2)
- added D16: 5V, LED_SMD:LED_0603_1608Metric, F.Cu at (91.0, 70.3)
- added D2: VIN, LED_SMD:LED_0603_1608Metric, F.Cu at (201.7, 70.5)
- added D7: 5V, LED_SMD:LED_0603_1608Metric, F.Cu at (184.4, 70.2)
- added D8: TVS 3V3, TXV_Library_Footprints:SOD882D, F.Cu at (356.5, 252.7)
- added D9: 3V3, LED_SMD:LED_0603_1608Metric, F.Cu at (359.0, 248.9)
- added J10: Debug, Connector_PinHeader_1.27mm:PinHeader_2x04_P1.27mm_Vertical_SMD, F.Cu at (175.2, 81.9)
- added J12: CAN1, Connector_JST:JST_GH_BM04B-GHS-TBT_1x04-1MP_P1.25mm_Vertical, B.Cu at (111.3, 59.8)
- added J13: CAN2, Connector_JST:JST_GH_BM04B-GHS-TBT_1x04-1MP_P1.25mm_Vertical, F.Cu at (104.5, 69.8)
- added J14: CAN1, Connector_JST:JST_GH_BM04B-GHS-TBT_1x04-1MP_P1.25mm_Vertical, F.Cu at (104.5, 59.8)
- added J15: CAN2, Connector_JST:JST_GH_BM04B-GHS-TBT_1x04-1MP_P1.25mm_Vertical, F.Cu at (111.3, 69.8)
- added J16: CAN1, Connector_JST:JST_GH_BM04B-GHS-TBT_1x04-1MP_P1.25mm_Vertical, F.Cu at (111.3, 59.8)
- added J17: CAN2, Connector_JST:JST_GH_BM04B-GHS-TBT_1x04-1MP_P1.25mm_Vertical, B.Cu at (111.3, 69.8)
- added J18: CAN1, Connector_JST:JST_GH_BM04B-GHS-TBT_1x04-1MP_P1.25mm_Vertical, B.Cu at (104.5, 59.8)
- added J19: CAN2, Connector_JST:JST_GH_BM04B-GHS-TBT_1x04-1MP_P1.25mm_Vertical, B.Cu at (104.5, 69.8)
- added J20: Cam0, TXV_Library_Footprints:Molex_Nano-Fit_105309-xx02_1x02_P2.50mm_Vertical, F.Cu at (93.0, 88.8)
- added J21: Cam1, TXV_Library_Footprints:Molex_Nano-Fit_105309-xx02_1x02_P2.50mm_Vertical, F.Cu at (101.4, 88.8)
- added J22: Cam2, TXV_Library_Footprints:Molex_Nano-Fit_105309-xx02_1x02_P2.50mm_Vertical, F.Cu at (109.8, 88.8)
- added J23: Payload, TXV_Library_Footprints:Molex_Nano-Fit_105309-xx02_1x02_P2.50mm_Vertical, F.Cu at (104.0, 80.5)
- added J9: Debug, Connector_PinHeader_2.54mm:PinHeader_1x08_P2.54mm_Vertical_SMD_Pin1Left, B.Cu at (160.6, 77.2)
- added L3: 4.7u, TXV_Library_Footprints:SRN4018TA-4R7M, F.Cu at (91.8, 81.2)
- added LED1: LED_Small_Filled, LED_SMD:LED_0603_1608Metric, F.Cu at (156.8, 72.5)
- added LED2: LED_Small_Filled, LED_SMD:LED_0603_1608Metric, F.Cu at (156.8, 74.1)
- added LS1: Speaker, TXV_Library_Footprints:Piezo_Buzzer, F.Cu at (150.1, 48.1)
- added R10: 1k, Resistor_SMD:R_0603_1608Metric, F.Cu at (198.5, 70.5)
- added R11: 120, Resistor_SMD:R_0603_1608Metric, F.Cu at (153.7, 72.5)
- added R13: 56k, Resistor_SMD:R_0603_1608Metric, F.Cu at (198.5, 68.8)
- added R16: 1k, Resistor_SMD:R_0603_1608Metric, F.Cu at (156.3, 46.6)
- added R17: 1k, Resistor_SMD:R_0603_1608Metric, F.Cu at (187.5, 70.2)
- added R28: 120, Resistor_SMD:R_0603_1608Metric, F.Cu at (115.5, 59.8)
- added R29: 120, Resistor_SMD:R_0603_1608Metric, F.Cu at (115.5, 69.8)
- added R30: 120, Resistor_SMD:R_0603_1608Metric, F.Cu at (355.8, 248.9)
- added R31: R, Resistor_SMD:R_0603_1608Metric, F.Cu at (119.4, 79.2)
- added R32: 120, Resistor_SMD:R_0603_1608Metric, F.Cu at (92.3, 95.8)
- added R33: 120, Resistor_SMD:R_0603_1608Metric, F.Cu at (100.8, 95.8)
- added R34: 120, Resistor_SMD:R_0603_1608Metric, F.Cu at (109.2, 95.8)
- added R35: 10k, Resistor_SMD:R_0603_1608Metric, F.Cu at (92.3, 97.4)
- added R36: 10k, Resistor_SMD:R_0603_1608Metric, F.Cu at (100.8, 97.4)
- added R37: 10k, Resistor_SMD:R_0603_1608Metric, F.Cu at (109.2, 97.4)
- added R38: 120, Resistor_SMD:R_0603_1608Metric, F.Cu at (92.3, 94.2)
- added R39: 120, Resistor_SMD:R_0603_1608Metric, F.Cu at (100.8, 94.2)
- added R40: 120, Resistor_SMD:R_0603_1608Metric, F.Cu at (109.2, 94.2)
- added R41: 10k, Resistor_SMD:R_0603_1608Metric, F.Cu at (191.5, 85.2)
- added R42: 10k, Resistor_SMD:R_0603_1608Metric, F.Cu at (191.5, 115.1)
- added R43: R, Resistor_SMD:R_0603_1608Metric, F.Cu at (94.0, 73.7)
- added R44: R, Resistor_SMD:R_0603_1608Metric, F.Cu at (91.0, 73.7)
- added R45: 1k, Resistor_SMD:R_0603_1608Metric, F.Cu at (94.0, 70.3)
- added R46: 10k, Resistor_SMD:R_0603_1608Metric, F.Cu at (94.0, 72.0)
- added R47: 10k, Resistor_SMD:R_0603_1608Metric, F.Cu at (91.0, 72.0)
- added U10: ICM-20602, Package_LGA:LGA-16_3x3mm_P0.5mm_LayoutBorder3x5y, F.Cu at (165.5, 76.2)
- added U11: LPS25HB, Package_LGA:ST_HLGA-10_2.5x2.5mm_P0.6mm_LayoutBorder3x2y, F.Cu at (175.3, 57.2)
- added U12: SFH617A-1X007T, Package_DIP:SMDIP-4_W9.53mm_Clearance8mm, F.Cu at (112.3, 78.9)
- added U13: TS30041, Package_DFN_QFN:QFN-16-1EP_3x3mm_P0.5mm_EP1.75x1.75mm_ThermalVias, F.Cu at (91.8, 76.7)
- added U6: W25Q256JV, TXV_Library_Footprints:WSON-8-8x6mm, F.Cu at (161.6, 52.5)
- added U7: MCP1700-3302E, Package_TO_SOT_SMD:SOT-23, F.Cu at (359.4, 254.0)
- added U8: MCP2562FDx-x_MF, Package_DFN_QFN:DFN-8-1EP_3x3mm_P0.65mm_EP1.55x2.4mm, F.Cu at (118.5, 59.8)
- added U9: MCP2562FDx-x_MF, Package_DFN_QFN:DFN-8-1EP_3x3mm_P0.65mm_EP1.55x2.4mm, F.Cu at (118.5, 69.8)
- added X1: TXC-7C, Oscillator:Oscillator_SMD_TXC_7C-4Pin_5.0x3.2mm, F.Cu at (179.4, 66.0)
- J2: footprint TXV_Library_Footprints:Molex_Nano-Fit_105309-xx02_1x02_P2.50mm_Vertical -> Connector_Molex:Molex_Mega-Fit_76825-0002_2x01_P5.70mm_Horizontal
- J5: footprint Connector_JST:JST_GH_BM04B-GHS-TBT_1x04-1MP_P1.25mm_Vertical -> Connector_JST:JST_XH_B4B-XH-A_1x04_P2.50mm_Vertical
- Q3, Q4: value BSZ0905PNSATMA1 -> SISA88DN or similar; footprint TXV_Library_Footprints:PG_TSDSON-8 -> TXV_Library_Footprints:PowerPAK_1212-8
- Q5, Q6: value BC817W -> SISA88DN or similar; footprint Package_TO_SOT_SMD:SOT-323_SC-70 -> TXV_Library_Footprints:PowerPAK_1212-8
- R12, R15: value 10k -> 120
- R14, R18: value 200 -> 10k
- U2: footprint Package_TO_SOT_SMD:SOT-23-6 -> Package_TO_SOT_SMD:SOT-23-5
- U5: value ECU -> STM32G491MET6-LQFP80; footprint TXV_Library_Footprints:ECU_Footprint_simple -> Package_QFP:LQFP-80_12x12mm_P0.5mm
- moved G1 168.9 mm to (337.7, 139.5)
- moved J2 99.1 mm to (265.4, 81.8)
- moved TH1 92.7 mm to (84.8, 33.0)
- moved R14 86.0 mm to (201.8, 68.8)
- moved J8 85.4 mm to (170.7, 122.5), turned to 180 degrees
- moved Q3 81.5 mm to (153.8, 58.8), turned to 90 degrees
- moved R15 79.2 mm to (156.4, 59.1), turned to -90 degrees
- moved J5 77.4 mm to (246.2, 65.3)
- moved R8 76.6 mm to (175.7, 67.1)
- moved J3 73.0 mm to (183.9, 121.8)
- moved Q4 73.0 mm to (89.0, 93.6), turned to 90 degrees
- moved R18 70.1 mm to (187.5, 71.8), turned to 180 degrees
- moved H1 69.0 mm to (174.0, 36.8)
- moved R19 67.9 mm to (184.4, 71.8), turned to 180 degrees
- moved Q5 66.0 mm to (97.3, 93.6), turned to 90 degrees
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Connections:
- net /Vbat renamed +BATT
- C15 pad 2: Net-(C15-Pad2) -> /Vin
- C16 pad 1: Net-(C15-Pad2) -> /Vin
- C8 pad 1: +3V3 -> Net-(C8-Pad1)
- D3 pad 1: /~ACOK -> /~{ACOK}
- D4 pad 1: /~CHGOK -> /~{CHGOK}
- J5 pad 1: (no net) -> unconnected-(J5-Pad1)
- J5 pad 2: /Cell2 -> unconnected-(J5-Pad2)
- J5 pad 3: /Cell1 -> unconnected-(J5-Pad3)
- J5 pad 4: GND -> unconnected-(J5-Pad4)
- Q3 pad 1: /Cell1 -> Net-(Q3-Pad1)
- Q3 pad 2: Net-(Q3-Pad2) -> Net-(LS1-Pad2)
- Q3 pad 3: Net-(Q3-Pad3) -> GND
- Q4 pad 1: /Cell2 -> Net-(Q4-Pad1)
- Q4 pad 2: Net-(Q4-Pad2) -> Net-(D13-Pad2)
- Q4 pad 3: Net-(Q4-Pad3) -> GND
- Q5 pad 2: GND -> Net-(D14-Pad2)
- Q5 pad 3: Net-(Q5-Pad3) -> GND
- Q6 pad 2: GND -> Net-(D15-Pad2)
- Q6 pad 3: Net-(Q6-Pad3) -> GND
- R12 pad 1: Net-(Q6-Pad1) -> /LED2
- R12 pad 2: Net-(R12-Pad2) -> Net-(LED2-Pad2)
- R14 pad 1: Net-(Q3-Pad2) -> /12V_Sense
- R14 pad 2: Net-(Q5-Pad3) -> GND
- R15 pad 1: /Cell1 -> /Speaker
- R15 pad 2: Net-(Q5-Pad3) -> Net-(Q3-Pad1)
- R18 pad 1: Net-(Q4-Pad2) -> +5V
- R18 pad 2: Net-(Q6-Pad3) -> /5V_Sense
- R19 pad 1: /Cell2 -> /5V_Sense
- R19 pad 2: Net-(Q6-Pad3) -> GND
- R22 pad 1: +3V3 -> Net-(C8-Pad1)
- R23 pad 1: +3V3 -> Net-(C8-Pad1)
- R24 pad 1: +3V3 -> Net-(C8-Pad1)
- R8 pad 1: Net-(Q5-Pad1) -> +3V3
- R8 pad 2: Net-(R12-Pad2) -> /NRST
- SW1 pad 3: (no net) -> unconnected-(SW1-Pad3)
- SW2 pad 3: (no net) -> unconnected-(SW2-Pad3)
- SW3 pad 3: GND -> Net-(SW3-Pad3)
- SW4 pad 3: GND -> Net-(SW4-Pad3)
- U1 pad 8: (no net) -> unconnected-(U1-Pad8)
- U3 pad 11: Net-(C15-Pad2) -> /Vin
- U3 pad 2: Net-(C15-Pad2) -> /Vin
- U3 pad 3: Net-(C15-Pad2) -> /Vin
- U3 pad 6: (no net) -> unconnected-(U3-Pad6)
- U3 pad 7: (no net) -> unconnected-(U3-Pad7)
- U3 pad 8: (no net) -> unconnected-(U3-Pad8)
- U3 pad 9: (no net) -> unconnected-(U3-Pad9)
- U4 pad 17: (no net) -> unconnected-(U4-Pad17)
- U4 pad 3: /~ACOK -> /~{ACOK}
- U4 pad 4: /~CHGOK -> /~{CHGOK}
- U4 pad 5: +3V3 -> Net-(C8-Pad1)
- U5 pad 17: +12V -> unconnected-(U5-Pad17)
- U5 pad 18: GND -> /BARO_SPI1_NSS
- U5 pad 19: +5V -> /BARO_SPI1_SCK
- U5 pad 26: (no net) -> unconnected-(U5-Pad26)
- U5 pad 27: Net-(R12-Pad2) -> GND
- U5 pad 28: (no net) -> +3V3
- U5 pad 29: GND -> +3V3
- U5 pad 30: /NTC -> unconnected-(U5-Pad30)
- U5 pad 31: Net-(Q3-Pad3) -> unconnected-(U5-Pad31)
- U5 pad 32: (no net) -> unconnected-(U5-Pad32)
- U5 pad 33: GND -> /QSPI1_CLK
- U5 pad 34: (no net) -> /QSPI1_BK1_NCS
- U5 pad 35: Net-(Q4-Pad3) -> /QSPI1_BK1_IO0
- U5 pad 36: (no net) -> /QSPI1_BK1_IO1
- U5 pad 37: GND -> /QSPI1_BK1_IO2
- U5 pad 38: (no net) -> /QSPI1_BK1_IO3
- U5 pad 39: /~CHGOK -> /Speaker
- U5 pad 40: (no net) -> GND
- U5 pad 41: GND -> +3V3
- U5 pad 42: (no net) -> unconnected-(U5-Pad42)
- U5 pad 43: /~ACOK -> unconnected-(U5-Pad43)
- U5 pad 44: (no net) -> unconnected-(U5-Pad44)
- U5 pad 45: GND -> unconnected-(U5-Pad45)
- U5 pad 46: (no net) -> unconnected-(U5-Pad46)
- U5 pad 47: /SUPPLY_CURRENT_SENSE -> unconnected-(U5-Pad47)
- U5 pad 48: (no net) -> unconnected-(U5-Pad48)
- U5 pad 49: GND -> unconnected-(U5-Pad49)
Routing:
- net /NTC: track 168.5 -> 0.00 mm, vias 3 -> 0
- net /SUPPLY_CURRENT_SENSE: track 138.0 -> 0.00 mm, vias 2 -> 0
- net +12V: track 135.2 -> 0.00 mm, vias 7 -> 4
- net /Cell1: track 98.1 -> 0.00 mm
- net /Cell2: track 97.8 -> 0.00 mm
- net /~CHGOK: track 93.8 -> 0.00 mm, vias 2 -> 0
- net /~ACOK: track 90.1 -> 0.00 mm, vias 2 -> 0
- net PYRO: track 87.5 -> 0.00 mm
- net Net-(Q4-Pad3): track 80.6 -> 0.00 mm
- net +5V: track 93.2 -> 14.2 mm
- net Net-(Q3-Pad3): track 71.6 -> 0.00 mm
- net Net-(R12-Pad2): track 47.6 -> 0.00 mm
- net +3V3: track 10.8 -> 31.0 mm
- net Net-(C15-Pad2): track 16.1 -> 0.00 mm, vias 7 -> 0
- net Net-(Q1-Pad2): track 46.2 -> 31.8 mm
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- added copper zone on B.Cu, net +BATT
- removed copper zone on B.Cu, net GND
- removed copper zone on F.Cu, net GND
- removed copper zone on B.Cu, net Net-(C15-Pad2)
- removed copper zone on F.Cu, net Net-(C15-Pad2)
Other:
- board size 118.5 x 100 mm -> 118.5 x 104.3 mm
- net class Default removed
- board text added: "PMU v2.0"
- board text removed: "BALANCE"
- board text removed: "BATT"
- board text removed: "ECU"
- board text removed: "PMU v1.0"
- board text removed: "PYRO"
- board text removed: "STM"
- board text removed: "Temp"
