File: uHoubolt_PCB_PMU.kicad_pcb (KiCad board)
At the start: 2 copper layers, 118.5 x 104.3 mm, 167 parts, among them J1 Umbilical, J10 Debug, J12 CAN1, J13 CAN2, J14 CAN1, J15 CAN2, J16 CAN1, J17 CAN2, J18 CAN1, J19 CAN2, J2 Battery, J20 Cam0, J21 Cam1, J22 Cam2, J23 Payload, J3 Power, J5 Batterycells, J8 12V, J9 Debug, Q1 BSZ0905PNSATMA1, Q2 BSZ0902NSATMA1, Q3 SISA88DN or similar, Q4 SISA88DN or similar, Q5 SISA88DN or similar, Q6 SISA88DN or similar, SW1 Power_1, SW2 Power_2, SW3 Pyro_1, SW4 Pyro_2, U1 LM5069, U10 ICM-20602, U11 LPS25HB, U12 SFH617A-1X007T, U13 TS30041, U2 LMP8640 F, U3 TS30041, U4 MP26123, U5 STM32G491MET6-LQFP80, U6 W25Q256JV, U7 MCP1700-3302E, U8 MCP2562FDx-x_MF, U9 MCP2562FDx-x_MF, X1 TXC-7C

Commit message: [WIP] PMUv2
Parts:
- added C49: 100n, Capacitor_SMD:C_0402_1005Metric, F.Cu at (177.6, 122.0)
- added C50: 22u, Capacitor_SMD:C_0805_2012Metric, F.Cu at (177.6, 123.5)
- added C51: 22u, Capacitor_SMD:C_0805_2012Metric, F.Cu at (177.6, 125.5)
- added C52: 22u, Capacitor_SMD:C_0805_2012Metric, F.Cu at (168.0, 138.5)
- added C53: 4.7u, Capacitor_SMD:C_0603_1608Metric, F.Cu at (173.0, 141.0)
- added C54: 4.7u, Capacitor_SMD:C_0603_1608Metric, F.Cu at (164.5, 138.0)
- added C55: 100n, Capacitor_SMD:C_0603_1608Metric, F.Cu at (167.5, 127.8)
- added C56: 100n, Capacitor_SMD:C_0402_1005Metric, F.Cu at (167.5, 130.5)
- added C57: 2.2n, Capacitor_SMD:C_0603_1608Metric, F.Cu at (174.0, 123.5)
- added C58: 2.2n, Capacitor_SMD:C_0603_1608Metric, F.Cu at (172.5, 123.5)
- added C59: 22u, Capacitor_SMD:C_0805_2012Metric, F.Cu at (170.0, 123.0)
- added C60: 22u, Capacitor_SMD:C_0805_2012Metric, F.Cu at (170.0, 127.0)
- added D17: OUT 1, LED_SMD:LED_0603_1608Metric, F.Cu at (128.0, 56.5)
- added D18: Shottky, Diode_SMD:D_SOD-123F, F.Cu at (125.5, 46.5)
- added D19: LED, LED_SMD:LED_0603_1608Metric, F.Cu at (172.0, 135.5)
- added D20: LED, LED_SMD:LED_0603_1608Metric, F.Cu at (173.5, 135.5)
- added D21: PMEG3050EP, Diode_SMD:D_SOD-128, F.Cu at (166.5, 135.5)
- added D22: PMEG3050EP, Diode_SMD:D_SOD-128, F.Cu at (160.0, 129.5)
- added J11: AltimaxPwr, TXV_Library_Footprints:Molex_SL_1x2_Vertical, F.Cu at (177.5, 118.8)
- added J24: Output, TXV_Library_Footprints:Molex_Nano-Fit_105309-xx02_1x02_P2.50mm_Vertical, F.Cu at (126.6, 50.1)
- added J25: RCU, TXV_Library_Footprints:Molex_SL_1x2_Vertical, F.Cu at (177.0, 81.5)
- added J26: Umbilical0, TXV_Library_Footprints:Molex_Nano-Fit_105309-xx02_1x02_P2.50mm_Vertical, B.Cu at (136.5, 155.0)
- added J4: BatteryAltimax, TXV_Library_Footprints:Molex_SL_1x2_Vertical, F.Cu at (168.5, 118.8)
- added J6: AltimaxArm, TXV_Library_Footprints:Molex_SL_1x2_Vertical, F.Cu at (191.0, 118.8)
- added J7: Umbilical1, TXV_Library_Footprints:Molex_Nano-Fit_105309-xx02_1x02_P2.50mm_Vertical, F.Cu at (167.5, 146.0)
- added JP1: Jumper_2_Open, Jumper:SolderJumper-2_P1.3mm_Open_RoundedPad1.0x1.5mm, F.Cu at (144.0, 141.4)
- added JP3: Jumper_2_Open, Jumper:SolderJumper-2_P1.3mm_Open_RoundedPad1.0x1.5mm, F.Cu at (187.0, 99.8)
- added JP4: Jumper_3_Open, Jumper:SolderJumper-3_P1.3mm_Open_RoundedPad1.0x1.5mm, F.Cu at (160.8, 50.2)
- added JP5: Jumper_3_Open, Jumper:SolderJumper-3_P1.3mm_Open_RoundedPad1.0x1.5mm, F.Cu at (150.5, 50.0)
- added JP6: Jumper_3_Open, Jumper:SolderJumper-3_P1.3mm_Open_RoundedPad1.0x1.5mm, F.Cu at (140.5, 50.0)
- added JP7: Jumper_3_Open, Jumper:SolderJumper-3_P1.3mm_Open_RoundedPad1.0x1.5mm, F.Cu at (130.5, 49.5)
- added JP8: Jumper_2_Open, Jumper:SolderJumper-2_P1.3mm_Open_RoundedPad1.0x1.5mm, F.Cu at (175.0, 131.0)
- added L4: 4.7u, TXV_Library_Footprints:SRN4018TA-4R7M, F.Cu at (164.5, 129.0)
- added Q7: SISA88DN or similar, TXV_Library_Footprints:PowerPAK_1212-8, F.Cu at (124.5, 54.5)
- added R48: 10k, Resistor_SMD:R_0603_1608Metric, F.Cu at (130.5, 55.5)
- added R49: 120, Resistor_SMD:R_0603_1608Metric, F.Cu at (128.0, 53.5)
- added R50: 10k, Resistor_SMD:R_0603_1608Metric, F.Cu at (175.5, 134.5)
- added R51: 120, Resistor_SMD:R_0603_1608Metric, F.Cu at (172.0, 138.5)
- added R52: 120, Resistor_SMD:R_0603_1608Metric, F.Cu at (173.5, 138.5)
- added R53: 750, Resistor_SMD:R_0603_1608Metric, F.Cu at (172.5, 126.5)
- added R54: 2.5k, Resistor_SMD:R_0603_1608Metric, F.Cu at (174.0, 126.5)
- added R55: 140m, Resistor_SMD:R_0805_2012Metric, F.Cu at (170.0, 125.0)
- added TH2: Thermistor_NTC, Connector_PinHeader_2.54mm:PinHeader_1x02_P2.54mm_Vertical, F.Cu at (176.5, 137.7)
- added U14: MP26123, Package_DFN_QFN:QFN-16-1EP_4x4mm_P0.65mm_EP2.15x2.15mm_ThermalVias, F.Cu at (171.0, 131.0)
- C15, C6: value 22u -> 100n; footprint Capacitor_SMD:C_0805_2012Metric -> Capacitor_SMD:C_0402_1005Metric
- C16, C5: value 100n -> 22u; footprint Capacitor_SMD:C_0402_1005Metric -> Capacitor_SMD:C_0805_2012Metric
- D11: value OUT 1 -> Shottky; footprint LED_SMD:LED_0603_1608Metric -> Diode_SMD:D_SOD-123F
- D14: value Shottky -> OUT 1; footprint Diode_SMD:D_SOD-123F -> LED_SMD:LED_0603_1608Metric
- J1: value Umbilical -> Umbilical0; moved to F.Cu
- J20: value Cam0 -> Output
- J21: value Cam1 -> Output
- J22: value Cam2 -> Output
- J8: value 12V -> RCU; moved to F.Cu
- R17: value 1k -> R
- R18: value 10k -> R
- R19: value 10k -> 1k
- R20, R21: value R -> 10k
- R33, R39: value 120 -> 10k
- R35, R37, R42: value 10k -> 120
- moved U7 316.2 mm to (85.8, 95.6), turned to 180 degrees
- moved C31 315.2 mm to (85.2, 98.1), turned to 0 degrees
- moved D9 311.8 mm to (85.2, 99.7), turned to 0 degrees
- moved D8 310.8 mm to (88.4, 95.4), turned to -90 degrees
- moved C36 309.0 mm to (88.4, 98.1), turned to 180 degrees
- moved R30 306.2 mm to (88.4, 99.7), turned to 180 degrees
- moved G1 282.9 mm to (56.2, 167.6)
- moved J5 163.2 mm to (99.8, 137.5)
- moved TH1 130.2 mm to (145.5, 148.1), turned to 0 degrees
- moved J2 125.7 mm to (152.5, 137.0)
- moved H2 123.4 mm to (71.0, 79.5)
- moved H1 120.8 mm to (71.0, 100.0)
- moved H4 117.8 mm to (54.5, 122.5)
- moved C42 107.8 mm to (86.9, 115.4), turned to 90 degrees
- moved C41 106.5 mm to (89.3, 117.8), turned to 180 degrees
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Connections:
- C15 pad 1: GND -> Net-(C15-Pad1)
- C15 pad 2: /Vin -> Net-(C15-Pad2)
- C16 pad 1: /Vin -> GND
- C16 pad 2: GND -> +5VP
- C17 pad 2: +5V -> +5VP
- C44 pad 2: +12V -> /Vin
- C45 pad 1: +12V -> /Vin
- C47 pad 2: +5VP -> +5V
- C48 pad 2: +5VP -> +5V
- C5 pad 1: Net-(C5-Pad1) -> GND
- C5 pad 2: Net-(C5-Pad2) -> +12V
- C6 pad 1: GND -> +12V
- C6 pad 2: +5V -> GND
- D11 pad 1: GND -> Net-(D11-Pad1)
- D13 pad 1: +5VP -> Net-(D13-Pad1)
- D14 pad 1: +5VP -> GND
- D15 pad 1: +5VP -> Net-(D15-Pad1)
- D3 pad 1: /~{ACOK} -> /BatteryCharger/~{ACOK}
- D4 pad 1: /~{CHGOK} -> /BatteryCharger/~{CHGOK}
- J20 pad 1: +5VP -> Net-(D11-Pad1)
- J20 pad 2: Net-(D13-Pad2) -> Net-(D11-Pad2)
- J21 pad 1: +5VP -> Net-(D13-Pad1)
- J21 pad 2: Net-(D14-Pad2) -> Net-(D13-Pad2)
- J22 pad 1: +5VP -> Net-(D15-Pad1)
- JP2 pad 1: Net-(JP2-Pad1) -> /Vcharge
- JP2 pad 2: GND -> /Vcharge1
- L1 pad 1: Net-(C5-Pad1) -> Net-(C15-Pad1)
- L1 pad 2: +5V -> +5VP
- L3 pad 2: +5VP -> +5V
- Q4 pad 2: Net-(D13-Pad2) -> Net-(D11-Pad2)
- Q5 pad 2: Net-(D14-Pad2) -> Net-(D13-Pad2)
- R17 pad 1: +5V -> Net-(R17-Pad1)
- R17 pad 2: Net-(D7-Pad2) -> +5VP
- R18 pad 1: +5V -> Net-(R17-Pad1)
- R18 pad 2: /5V_Sense -> GND
- R19 pad 1: /5V_Sense -> +5VP
- R19 pad 2: GND -> Net-(D7-Pad2)
- R20 pad 1: Net-(R20-Pad1) -> +5VP
- R20 pad 2: +5V -> /5VP_Sense
- R21 pad 1: Net-(R20-Pad1) -> /5VP_Sense
- R22 pad 2: /NTC -> /BatteryCharger/NTC
- R32 pad 1: /Cam0 -> /Out0
- R33 pad 1: /Cam1 -> GND
- R33 pad 2: Net-(D11-Pad2) -> /Out0
- R34 pad 1: /Cam2 -> /Out0
- R34 pad 2: Net-(D12-Pad2) -> Net-(Q4-Pad1)
- R35 pad 1: GND -> /Out1
- R35 pad 2: /Cam0 -> Net-(D12-Pad2)
- R36 pad 2: /Cam1 -> /Out1
- R37 pad 1: GND -> /Out1
- R37 pad 2: /Cam2 -> Net-(Q5-Pad1)
- R38 pad 1: /Cam0 -> /Out2
- R38 pad 2: Net-(Q4-Pad1) -> Net-(D14-Pad2)
- R39 pad 1: /Cam1 -> GND
- R39 pad 2: Net-(Q5-Pad1) -> /Out2
- R40 pad 1: /Cam2 -> /Out2
- R42 pad 1: Net-(SW4-Pad3) -> /Out3
- R42 pad 2: GND -> Net-(D17-Pad2)
- R43 pad 2: +5VP -> +5V
- R45 pad 1: +5VP -> +5V
- R46 pad 1: +5VP -> +5V
- R46 pad 2: /5VP_Sense -> /5V_Sense
- R47 pad 1: /5VP_Sense -> /5V_Sense
- SW2 pad 1: GND -> +7.4V
- SW2 pad 2: Net-(Q1-Pad2) -> Net-(SW2-Pad2)
- SW3 pad 2: Net-(SW3-Pad2) -> PYRO
- SW4 pad 1: Net-(SW3-Pad2) -> Net-(SW4-Pad1)
- SW4 pad 2: PYRO -> Net-(SW4-Pad2)
- SW4 pad 3: Net-(SW4-Pad3) -> unconnected-(SW4-Pad3)
- TH1 pad 1: /NTC -> /BatteryCharger/NTC
- U13 pad 11: +12V -> /Vin
- U13 pad 2: +12V -> /Vin
- U13 pad 3: +12V -> /Vin
- U3 pad 1: Net-(C5-Pad1) -> Net-(C15-Pad1)
- U3 pad 10: Net-(C5-Pad2) -> Net-(C15-Pad2)
- U3 pad 11: /Vin -> +12V
- U3 pad 12: Net-(C5-Pad1) -> Net-(C15-Pad1)
- U3 pad 13: Net-(C5-Pad1) -> Net-(C15-Pad1)
- U3 pad 16: Net-(C5-Pad1) -> Net-(C15-Pad1)
- U3 pad 2: /Vin -> +12V
- U3 pad 3: /Vin -> +12V
- U3 pad 5: Net-(R20-Pad1) -> Net-(R17-Pad1)
- U4 pad 2: /NTC -> /BatteryCharger/NTC
- U4 pad 3: /~{ACOK} -> /BatteryCharger/~{ACOK}
- U4 pad 4: /~{CHGOK} -> /BatteryCharger/~{CHGOK}
- U4 pad 7: Net-(JP2-Pad1) -> Net-(JP1-Pad1)
- U5 pad 14: /BARO_INT -> unconnected-(U5-Pad14)
- U5 pad 17: unconnected-(U5-Pad17) -> /BARO_INT
- U5 pad 52: /Cam0 -> /Out0
- U5 pad 53: /Cam1 -> /Out1
- U5 pad 54: /Cam2 -> /Out2
- U5 pad 55: /Payload -> /Out3
Routing:
- net +3V3: track 31.0 -> 61.8 mm
- net Net-(SW3-Pad2): track 29.7 -> 0.00 mm
- net Net-(Q1-Pad2): track 31.8 -> 3.71 mm
- net GND: track 44.1 -> 65.3 mm, vias 12 -> 3
- net /QSPI1_CLK: track 0.00 -> 15.7 mm, vias 0 -> 2
- net Net-(LS1-Pad2): track 0.00 -> 15.7 mm
- net +5V: track 14.2 -> 0.00 mm
- net /Vcharge: track 13.7 -> 0.00 mm
- net /QSPI1_BK1_IO0: track 0.00 -> 13.4 mm, vias 0 -> 2
- net +BATT: track 11.8 -> 0.00 mm, vias 2 -> 0
- net Net-(L2-Pad2): track 10.3 -> 0.00 mm, vias 2 -> 0
- net /Vin: track 20.6 -> 11.0 mm, vias 7 -> 0
- net /QSPI1_BK1_IO3: track 0.00 -> 8.93 mm
- net Net-(C5-Pad1): track 7.72 -> 0.00 mm
- net /BARO_INT: track 0.00 -> 7.52 mm, vias 0 -> 2
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- removed copper zone on F.Cu, net +5V
- removed copper zone on B.Cu, net +BATT
- removed copper zone on F.Cu, net +BATT
- removed copper zone on F.Cu, net /Vcharge
- removed copper zone on F.Cu, net Net-(C11-Pad1)
- removed copper zone on F.Cu, net Net-(C5-Pad1)
- removed copper zone on F.Cu, net Net-(L2-Pad2)
Other:
- board size 118.5 x 104.3 mm -> 118 x 118 mm
- board text removed: "12V"
- board text removed: "Charger"
- board text removed: "GND"
