File: uHoubolt_PCB_PMU.kicad_pcb (KiCad board)
At the start: 4 copper layers, 118 x 118 mm, 166 parts, among them J1 Umbilical0, J10 Debug, J11 AltimaxPwr, J12 CAN1, J13 CAN2, J14 CAN1, J15 CAN2, J16 CAN1, J17 CAN2, J18 CAN1, J19 CAN2, J2 Battery, J20 Output, J21 Output, J22 Output, J23 Payload, J24 Output, J25 RCU, J26 Umbilical0, J3 Power, J4 BatteryAltimax, J6 AltimaxArm, J7 Umbilical1, J8 RCU, J9 Debug, Q1 BSZ0905PNSATMA1, Q2 BSZ0902NSATMA1, Q3 SISA88DN or similar, Q4 SISA88DN or similar, Q5 SISA88DN or similar, Q6 SISA88DN or similar, Q7 SISA88DN or similar, SW1 Power_1, SW2 Power_2, SW3 Pyro_1, SW4 Pyro_2, U1 LM5069, U10 ICM-20602, U11 LPS25HB, U12 SFH617A-1X007T, U13 TS30041, U14 LiIon_Charger, U2 LMP8640 F, U3 TS30041, U4 LiIon_Charger, U5 STM32G491MET6-LQFP80, U6 W25Q256JV, U7 MCP1700-3302E, U8 MCP2562FDx-x_MF, U9 MCP2562FDx-x_MF, X1 TXC-7C

Commit message: PMU V3 "ready to order?"
ready to validate changes
Parts:
- removed J1, J26: Umbilical0, TXV_Library_Footprints:Molex_Nano-Fit_105309-xx02_1x02_P2.50mm_Vertical
- removed J7: Umbilical1, TXV_Library_Footprints:Molex_Nano-Fit_105309-xx02_1x02_P2.50mm_Vertical
- added D3: Pyro, LED_SMD:LED_0603_1608Metric, F.Cu at (120.5, 130.7)
- added D4: TVS 3V3, TXV_Library_Footprints:SOD882D, F.Cu at (142.1, 69.2)
- added J27: Umbilical0, TXV_Library_Footprints:Molex_MicroFit_2Pin_Vertical, F.Cu at (168.3, 60.0)
- added J28: Umbilical0, TXV_Library_Footprints:Molex_MicroFit_2Pin_Vertical, F.Cu at (165.2, 72.8)
- added J29: AltimaxArm, TXV_Library_Footprints:Molex_Nano-Fit_105309-xx02_1x02_P2.50mm_Vertical, F.Cu at (175.3, 68.6)
- added J5: Umbilical1, TXV_Library_Footprints:Molex_MicroFit_2Pin_Vertical, F.Cu at (183.5, 126.7)
- added R22: R, Resistor_SMD:R_0603_1608Metric, F.Cu at (180.1, 81.5)
- added R23: 1k, Resistor_SMD:R_0603_1608Metric, F.Cu at (120.5, 133.7)
- added R24: 56k, Resistor_SMD:R_0603_1608Metric, F.Cu at (122.0, 133.7)
- added R25: 10k, Resistor_SMD:R_0603_1608Metric, F.Cu at (122.0, 130.7)
- added R26: 10k, Resistor_SMD:R_0603_1608Metric, F.Cu at (140.8, 67.9)
- added R27: 56k, Resistor_SMD:R_0603_1608Metric, F.Cu at (140.8, 71.0)
- added U15: SFH617A-1X007T, Package_DIP:SMDIP-4_W9.53mm_Clearance8mm, F.Cu at (176.5, 79.2)
- D10, D12, D14, D17: value OUT 1 -> OUT
- D25: value OUT 1 -> Payload
- J8: value RCU -> Altimax_PWR
- moved J25 49.3 mm to (121.2, 72.0)
- moved J8 49.3 mm to (121.2, 65.0)
- moved U4 47.6 mm to (142.8, 67.7), turned to 90 degrees
- moved C43 44.4 mm to (126.2, 74.2), turned to -90 degrees
- moved C4 39.9 mm to (126.3, 70.6)
- moved R9 37.3 mm to (128.2, 72.3)
- moved C3 36.7 mm to (129.9, 73.5)
- moved C1 35.6 mm to (128.2, 69.1), turned to 90 degrees
- moved Q2 33.1 mm to (130.3, 67.9), turned to 90 degrees
- moved C19 31.2 mm to (129.8, 64.8), turned to 180 degrees
- moved U1 27.7 mm to (133.7, 71.8), turned to 180 degrees
- moved R6 25.9 mm to (132.8, 66.7), turned to -90 degrees
- moved U2 25.7 mm to (133.1, 62.5), turned to 180 degrees
- moved R7 25.0 mm to (134.7, 68.3), turned to 90 degrees
- moved R4 22.0 mm to (137.0, 67.5), turned to 0 degrees
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Connections:
- U4 pad 3: unconnected-(U4-Pad3) -> /~{EN}
- U4 pad 5: unconnected-(U4-Pad5) -> /~{CHGOK}
- U4 pad 6: unconnected-(U4-Pad6) -> /~{ACOK}
- U4 pad 8: unconnected-(U4-Pad8) -> /NTC
- U5 pad 10: unconnected-(U5-Pad10) -> /Battery_Sense
- U5 pad 14: unconnected-(U5-Pad14) -> /NTC
- U5 pad 32: unconnected-(U5-Pad32) -> /SUPPLY_CURRENT_SENSE
- U5 pad 49: unconnected-(U5-Pad49) -> /Pyro_Sense
- U5 pad 58: /SUPPLY_CURRENT_SENSE -> /~{EN}
Routing:
- net /NTC: track 0.00 -> 97.3 mm, vias 0 -> 2
- net /~{ACOK}: track 0.00 -> 79.7 mm, vias 0 -> 2
- net /~{CHGOK}: track 0.00 -> 76.0 mm, vias 0 -> 2
- net /~{EN}: track 0.00 -> 66.5 mm, vias 0 -> 2
- net /Battery_Sense: track 0.00 -> 64.5 mm, vias 0 -> 2
- net +5V: track 191.4 -> 146.7 mm
- net /Pyro_Sense: track 0.00 -> 42.7 mm
- net GND: track 62.0 -> 27.3 mm, vias 604 -> 181
- net Net-(J4-Pad1): track 6.29 -> 37.4 mm
- net PYRO: track 146.3 -> 172.4 mm, vias 1 -> 0
- net Net-(Q1-Pad2): track 38.3 -> 60.1 mm, vias 1 -> 0
- net /Vcharge: track 72.4 -> 51.9 mm, vias 0 -> 1
- net +12V: track 32.3 -> 14.2 mm, vias 7 -> 10
- net +3V3: track 132.5 -> 116.6 mm, vias 22 -> 23
- net /Out3: track 77.5 -> 61.8 mm
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- added copper zone on F.Cu, net +BATT
- added copper zone on F.Cu, net Net-(R17-Pad1)
- removed copper zone on F.Cu, net (none)
- removed copper zone on B.Cu, net /Vcharge
- removed copper zone on F.Cu, net Net-(R2-Pad2)
- removed copper zone on F.Cu, net Net-(R5-Pad2)
Other:
- board text removed: "C"
- board text removed: "JLCJLCJLCJLC"
- board text removed: "S"

Commit message: PMU Ready for check
Ready for conformity check
Routing:
- net PYRO: track 172.4 -> 171.7 mm
- net GND: vias 181 -> 184
