File: BatteryCharger.kicad_sch (KiCad schematic)
At the start: 23 parts, among them U4 MP26123

Commit message: [WIP] PMUv2
Parts:
- renumbered C7 to C52, C8 to C53, C9 to C54, C10 to C55, C11 to C56, C12 to C57, C13 to C58, C14 to C59, C18 to C60, D3 to D19, D4 to D20, D5 to D21, D6 to D22, JP1 to JP8, L2 to L4, R22 to R50, R23 to R51, R24 to R52, R25 to R53, R26 to R54, R27 to R55, TH1 to TH2, U4 to U14

Commit message: PMU v2 WIP
Parts:
- added D23: PMEG3050EP, Diode_SMD:D_SOD-128, symbol Device:D_Schottky
- added F2: Fuse_Small, Resistor_SMD:R_0805_2012Metric_Pad1.20x1.40mm_HandSolder, symbol Device:Fuse_Small
- renumbered C55 to C10, C56 to C11, C57 to C12, C58 to C13, C59 to C14, C60 to C18, C52 to C7, C53 to C8, C54 to C9, D19 to D3, D20 to D4, D21 to D5, D22 to D6, JP8 to JP1, L4 to L2, R50 to R22, R51 to R23, R52 to R24, R53 to R25, R54 to R26, R55 to R27, TH2 to TH1, U14 to U4
Connections:
- net Charger: now also F2.1; no longer C7.1, D5.2 (A), U4.1 (VCC)
- new net: C7.1, D23.1 (K), D5.2 (A), U4.1 (VCC)
- new net: D23.2 (A), F2.2
Other:
- moved on the sheet: C8
