File: uHoubolt_PCB_PMU.kicad_sch (KiCad schematic)
At the start: 167 parts, among them J1 Umbilical, J10 Debug, J12 CAN1, J13 CAN2, J14 CAN1, J15 CAN2, J16 CAN1, J17 CAN2, J18 CAN1, J19 CAN2, J2 Battery, J20 Cam0, J21 Cam1, J22 Cam2, J23 Payload, J3 Power, J5 Batterycells, J8 12V, J9 Debug, Q1 BSZ0905PNSATMA1, Q2 BSZ0902NSATMA1, Q3 SISA88DN or similar, Q4 SISA88DN or similar, Q5 SISA88DN or similar, Q6 SISA88DN or similar, SW1 Power_1, SW2 Power_2, SW3 Pyro_1, SW4 Pyro_2, U1 LM5069, U10 ICM-20602, U11 LPS25HB, U12 SFH617A-1X007T, U13 TS30041, U2 LMP8640 F, U3 TS30041, U4 MP26123, U5 STM32G491MET6-LQFP80, U6 W25Q256JV, U7 MCP1700-3302E, U8 MCP2562FDx-x_MF, U9 MCP2562FDx-x_MF, X1 TXC-7C

Commit message: [WIP] Fixed References and Preps for PMUv2
Parts:
- removed C10: 100n, Capacitor_SMD:C_0603_1608Metric, symbol uHoubolt_PCB_PMU-rescue:C_Small-Device
- removed C11: 100n, Capacitor_SMD:C_0402_1005Metric, symbol uHoubolt_PCB_PMU-rescue:C_Small-Device
- removed C12, C13: 2.2n, Capacitor_SMD:C_0603_1608Metric, symbol uHoubolt_PCB_PMU-rescue:C_Small-Device
- removed C14, C18, C7: 22u, Capacitor_SMD:C_0805_2012Metric, symbol uHoubolt_PCB_PMU-rescue:C_Small-Device
- removed C8, C9: 4.7u, Capacitor_SMD:C_0603_1608Metric, symbol uHoubolt_PCB_PMU-rescue:C_Small-Device
- removed D3, D4: LED, LED_SMD:LED_0603_1608Metric, symbol uHoubolt_PCB_PMU-rescue:LED-Device
- removed D5: PMEG3050EP, Diode_SMD:D_SOD-128, symbol uHoubolt_PCB_PMU-rescue:D_Schottky-Device
- removed D6: PMEG3050EP, Diode_SMD:D_SOD-128, symbol uHoubolt_PCB_PMU-rescue:D_Schottky_Small-Device
- removed JP2: Jumper_2_Open, Jumper:SolderJumper-2_P1.3mm_Open_RoundedPad1.0x1.5mm, symbol uHoubolt_PCB_PMU-rescue:Jumper_NO_Small-Device
- removed L2: 4.7u, TXV_Library_Footprints:SRN4018TA-4R7M, symbol uHoubolt_PCB_PMU-rescue:L-Device
- removed R22: 10k, Resistor_SMD:R_0603_1608Metric, symbol uHoubolt_PCB_PMU-rescue:R-Device
- removed R23, R24: 120, Resistor_SMD:R_0603_1608Metric, symbol uHoubolt_PCB_PMU-rescue:R_Small-Device
- removed R25: 750, Resistor_SMD:R_0603_1608Metric, symbol uHoubolt_PCB_PMU-rescue:R_Small-Device
- removed R26: 2.5k, Resistor_SMD:R_0603_1608Metric, symbol uHoubolt_PCB_PMU-rescue:R_Small-Device
- removed R27: 140m, Resistor_SMD:R_0805_2012Metric, symbol uHoubolt_PCB_PMU-rescue:R_Small-Device
- removed R42: 10k, Resistor_SMD:R_0603_1608Metric, symbol Device:R_Small
- removed TH1: Thermistor_NTC, Connector_PinHeader_2.54mm:PinHeader_1x02_P2.54mm_Vertical, symbol Sensor_Temperature:KT100
- removed U4: MP26123, Package_DFN_QFN:QFN-16-1EP_4x4mm_P0.65mm_EP2.15x2.15mm_ThermalVias, symbol TXV_Library_Symbols:MP26123
- C1, C15, C16, C17, C19, C3, C44, C45, C46, C47, C48, C5, C6: symbol uHoubolt_PCB_PMU-rescue:C-Device -> Device:C
- C4, C43: symbol uHoubolt_PCB_PMU-rescue:CP-Device -> Device:C_Polarized
- D1: symbol uHoubolt_PCB_PMU-rescue:D_TVS-Device -> Device:D_TVS
- H1, H2, H3, H4: symbol uHoubolt_PCB_PMU-rescue:MountingHole_Pad-Mechanical -> Mechanical:MountingHole_Pad
- J1, J2, J8: symbol uHoubolt_PCB_PMU-rescue:Conn_01x02-Connector_Generic -> Connector_Generic:Conn_01x02
- J3: symbol uHoubolt_PCB_PMU-rescue:Conn_01x03-Connector_Generic -> Connector_Generic:Conn_01x03
- L1, L3: symbol uHoubolt_PCB_PMU-rescue:L-Device -> Device:L
- Q1: symbol uHoubolt_PCB_PMU-rescue:Q_PMOS_SGD-Device -> Device:Q_PMOS_SGD
- R1: symbol uHoubolt_PCB_PMU-rescue:R_Small-Device -> Device:R_Small
- R2, R20, R21, R3, R4, R43, R44, R5, R6, R7, R9: symbol uHoubolt_PCB_PMU-rescue:R-Device -> Device:R
- SW1, SW2, SW3, SW4: symbol uHoubolt_PCB_PMU-rescue:SW_Push_SPDT-Switch -> Switch:SW_Push_SPDT
Connections:
- net BARO_INT: now also U5.17 (PA3); no longer U5.14 (PA2)
- net GND: no longer SW2.1 (A)
- net PYRO: now also SW3.2 (B); no longer SW4.2 (B)
- net Vcharge: no longer J1.1 (Pin_1)
- net at Q1.2 (G), R1.2, SW1.2 (B): no longer SW2.2 (B)
- net at SW4.1 (A): no longer SW3.2 (B)
- new net BatteryCharger/Charger: J1.1 (Pin_1)
- no-connect marks 40 -> 38
Other:
- added sheet BatteryCharger (BatteryCharger.kicad_sch)
- added sheet Output0 (Output.kicad_sch)
- added sheet Output1 (Output.kicad_sch)
- added sheet Output2 (Output.kicad_sch)
- added sheet Output3 (Output.kicad_sch)
- note removed: "I_charge = 200mV / RS1 RS1 = 200mV / I_charge"
- moved on the sheet: J5, SW1, SW2, SW4

Commit message: [WIP] PMUv2
Parts:
- removed C15, C17, C44, C47, C48, C6: 22u, Capacitor_SMD:C_0805_2012Metric, symbol Device:C
- removed C16, C45, C46, C5: 100n, Capacitor_SMD:C_0402_1005Metric, symbol Device:C
- removed D10, D11, D12: OUT 1, LED_SMD:LED_0603_1608Metric, symbol Device:LED_Small_Filled
- removed D13, D14, D15: Shottky, Diode_SMD:D_SOD-123F, symbol Device:D_Schottky_Small_Filled
- removed D16, D7: 5V, LED_SMD:LED_0603_1608Metric, symbol Device:LED_Small_Filled
- removed J20: Cam0, TXV_Library_Footprints:Molex_Nano-Fit_105309-xx02_1x02_P2.50mm_Vertical, symbol Connector_Generic:Conn_01x02
- removed J21: Cam1, TXV_Library_Footprints:Molex_Nano-Fit_105309-xx02_1x02_P2.50mm_Vertical, symbol Connector_Generic:Conn_01x02
- removed J22: Cam2, TXV_Library_Footprints:Molex_Nano-Fit_105309-xx02_1x02_P2.50mm_Vertical, symbol Connector_Generic:Conn_01x02
- removed L1, L3: 4.7u, TXV_Library_Footprints:SRN4018TA-4R7M, symbol Device:L
- removed Q4, Q5, Q6: SISA88DN or similar, TXV_Library_Footprints:PowerPAK_1212-8, symbol Device:Q_NMOS_GDS
- removed R17, R45: 1k, Resistor_SMD:R_0603_1608Metric, symbol Device:R_Small
- removed R18, R19, R35, R36, R37, R46, R47: 10k, Resistor_SMD:R_0603_1608Metric, symbol Device:R_Small
- removed R20, R21, R43, R44: R, Resistor_SMD:R_0603_1608Metric, symbol Device:R
- removed R32, R33, R34, R38, R39, R40: 120, Resistor_SMD:R_0603_1608Metric, symbol Device:R_Small
- removed U13, U3: TS30041, Package_DFN_QFN:QFN-16-1EP_3x3mm_P0.5mm_EP1.75x1.75mm_ThermalVias, symbol TXV_Library_Symbols:TS30041
- added C49: 100n, Capacitor_SMD:C_0402_1005Metric, symbol Device:C
- added C50, C51: 22u, Capacitor_SMD:C_0805_2012Metric, symbol Device:C_Polarized
- added J11: AltimaxPwr, TXV_Library_Footprints:Molex_SL_1x2_Vertical, symbol Connector_Generic:Conn_01x02
- added J25: RCU, TXV_Library_Footprints:Molex_SL_1x2_Vertical, symbol Connector_Generic:Conn_01x02
- added J26: Umbilical0, TXV_Library_Footprints:Molex_Nano-Fit_105309-xx02_1x02_P2.50mm_Vertical, symbol Connector_Generic:Conn_01x02
- added J4: BatteryAltimax, TXV_Library_Footprints:Molex_SL_1x2_Vertical, symbol Connector_Generic:Conn_01x02
- added J6: AltimaxArm, TXV_Library_Footprints:Molex_SL_1x2_Vertical, symbol Connector_Generic:Conn_01x02
- added J7: Umbilical1, TXV_Library_Footprints:Molex_Nano-Fit_105309-xx02_1x02_P2.50mm_Vertical, symbol Connector_Generic:Conn_01x02
- added JP2, JP3: Jumper_2_Open, Jumper:SolderJumper-2_P1.3mm_Open_RoundedPad1.0x1.5mm, symbol Jumper:SolderJumper_2_Open
- J1: value Umbilical -> Umbilical0
- J8: value 12V -> RCU
Connections:
- net BatteryCharger/Charger is gone; now on net Vcharge: J1.1 (Pin_1)
- net +12V: now also J25.1 (Pin_1)
- net GND: now also J25.2 (Pin_2), J26.2 (Pin_2), JP3.1 (A)
- net Payload: no longer U5.55 (PC9)
- net Vcharge: now also J26.1 (Pin_1), JP2.1 (A)
- net +7.4V: now reaches SW2.1 (A)
- net +7.4V: now also J4.1 (Pin_1)
- net at SW2.2 (B): now also C49.1, C50.1, C51.1, J11.1 (Pin_1)
- net at SW4.1 (A): now also J6.2 (Pin_2)
- net at SW4.2 (B): now also J6.1 (Pin_1)
- net Cam0 renamed Out0
- net Cam1 renamed Out1
- net Cam2 renamed Out2
- new net GND1: C49.2, C50.2, C51.2, J11.2 (Pin_2), J4.2 (Pin_2), J7.2 (Pin_2), JP3.2 (B)
- new net Out3: U5.55 (PC9)
- new net Vcharge1: J7.1 (Pin_1), JP2.2 (B)
- no-connect marks 38 -> 36
Other:
- added sheet 5V (5V_SMPS.kicad_sch)
- added sheet 5VP (5V_SMPS.kicad_sch)
- added sheet BatteryCharger1 (BatteryCharger.kicad_sch)
- sheet Output0 ports: added Control; removed none
- sheet Output1 ports: added Control; removed none
- sheet Output2 ports: added Control; removed none
- sheet Output3 ports: added Control; removed none
- note added: "Outputs"
- note removed: "Akkulader 5V Buck STM 2x CAN Beeper 2-4x 5V/Bat High Side switch"
- note removed: "Cameras"
- moved on the sheet: C1, C19, C2, C20, C21, C22, C23, C24, C25, C26, C27, C28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

Commit message: PMU v2 WIP
Parts:
- removed C49: 100n, Capacitor_SMD:C_0402_1005Metric, symbol Device:C
- removed C50, C51: 22u, Capacitor_SMD:C_0805_2012Metric, symbol Device:C_Polarized
- removed J5: Batterycells, Connector_JST:JST_XH_B4B-XH-A_1x04_P2.50mm_Vertical, symbol Connector_Generic:Conn_01x04
- added F1: Fuse_Small, Resistor_SMD:R_0805_2012Metric_Pad1.20x1.40mm_HandSolder, symbol Device:Fuse_Small
- J2: footprint Connector_Molex:Molex_Mega-Fit_76825-0002_2x01_P5.70mm_Horizontal -> TXV_Library_Footprints:Molex_MegaFit_1x03_Vertical; symbol Connector_Generic:Conn_01x02 -> Connector_Generic:Conn_01x03
Connections:
- net Payload: now also U5.9 (PC1)
- net Vin: now also F1.1
- net +7.4V renamed BatteryCharger1/Battery
- net GND1 renamed GND_Altimax
- new net 5V/Input: F1.2
- no-connect marks 36 -> 32
Other:
- note added: "C:\Program Files\KiCad\6.0\share\kicad\symbols\"
- moved on the sheet: J11, J4, J7, JP2, JP3, SW2

Commit message: PMU V2 "ready to order"?
Parts:
- added D25: OUT 1, LED_SMD:LED_0603_1608Metric, symbol Device:LED_Small_Filled
- added R56: 120, Resistor_SMD:R_0603_1608Metric, symbol Device:R_Small
Connections:
- net GND: now also D25.1 (K)
- net Payload: now also R56.1
- net NTC: no longer names the net of U5.8 (PC0)
- new net: D25.2 (A), R56.2
- no-connect marks 32 -> 33
Changed lines of the file:
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@@
   (junction (at 121.285 69.215) (diameter 0) (color 0 0 0 0)
   )
+  (junction (at 151.765 146.685) (diameter 0) (color 0 0 0 0)
+  )
   (junction (at 141.605 57.785) (diameter 0) (color 0 0 0 0)
   )
@@
   (no_connect (at 66.04 266.065))
   (no_connect (at 66.04 337.185))
+  (no_connect (at 109.22 332.105))
   (wire (pts (xy 224.79 196.85) (xy 224.79 194.31))
     (stroke (width 0) (type default) (color 0 0 0 0))
@@
     (stroke (width 0) (type default) (color 0 0 0 0))
   )
+  (wire (pts (xy 151.765 152.4) (xy 151.765 153.035))
+    (stroke (width 0) (type default) (color 0 0 0 0))
+  )
   (wire (pts (xy 212.725 317.5) (xy 208.915 317.5))
     (stroke (width 0) (type default) (color 0 0 0 0))
@@
     (stroke (width 0) (type default) (color 0 0 0 0))
   )
-  (wire (pts (xy 118.745 332.105) (xy 109.22 332.105))
-    (stroke (width 0) (type default) (color 0 0 0 0))
-  )
   (wire (pts (xy 82.55 183.515) (xy 82.55 179.705))
     (stroke (width 0) (type default) (color 0 0 0 0))
@@
     (stroke (width 0) (type default) (color 0 0 0 0))
   )
-  (wire (pts (xy 146.685 146.685) (xy 154.94 146.685))
+  (wire (pts (xy 142.24 146.685) (xy 151.765 146.685))
     (stroke (width 0) (type default) (color 0 0 0 0))
   )
@@
     (stroke (width 0) (type default) (color 0 0 0 0))
   )
+  (wire (pts (xy 151.765 158.75) (xy 151.765 158.115))
+    (stroke (width 0) (type default) (color 0 0 0 0))
+  )
   (wire (pts (xy 99.695 111.76) (xy 99.695 115.57))
     (stroke (width 0) (type default) (color 0 0 0 0))
@@
     (stroke (width 0) (type default) (color 0 0 0 0))
   )
+  (wire (pts (xy 151.765 146.685) (xy 154.94 146.685))
+    (stroke (width 0) (type default) (color 0 0 0 0))
+  )
   (wire (pts (xy 240.03 323.85) (xy 240.03 323.215))
     (stroke (width 0) (type default) (color 0 0 0 0))
@@
     (stroke (width 0) (type default) (color 0 0 0 0))
   )
+  (wire (pts (xy 151.765 147.32) (xy 151.765 146.685))
+    (stroke (width 0) (type default) (color 0 0 0 0))
+  )
   (polyline (pts (xy 138.43 290.195) (xy 259.08 290.195))
     (stroke (width 0) (type default) (color 0 0 0 0))
@@
     (effects (font (size 1.27 1.27)) (justify left bottom))
   )
-  (label "Payload" (at 146.685 146.685 0)
+  (label "Payload" (at 142.24 146.685 0)
     (effects (font (size 1.27 1.27)) (justify left bottom))
   )
@@
     (effects (font (size 1.27 1.27)) (justify left bottom))
   )
-  (label "NTC" (at 118.745 332.105 180)
-    (effects (font (size 1.27 1.27)) (justify right bottom))
-  )
   (label "QSPI1_BK1_IO1" (at 124.46 268.605 180)
     (effects (font (size 1.27 1.27)) (justify right bottom))
@@
     (pin "1")
   )
+  (symbol (lib_id "Device:R_Small") (at 151.765 149.86 0) (unit 1)
+    (in_bom yes) (on_board yes)
+    (property "Reference" "R56" (id 0) (at 148.59 149.225 0))
+    (property "Value" "120" (id 1) (at 148.59 151.13 0))
+    (property "Footprint" "Resistor_SMD:R_0603_1608Metric" (id 2) (at 151.765 149.86 0)
+      (effects (font (size 1.27 1.27)) hide)
+    )
+    (property "Datasheet" "~" (id 3) (at 151.765 149.86 0)
+      (effects (font (size 1.27 1.27)) hide)
+    )
+    (pin "1")
+    (pin "2")
+  )
+  (symbol (lib_id "power:GND") (at 151.765 158.75 0) (unit 1)
+    (in_bom yes) (on_board yes)
+    (property "Reference" "#PWR022" (id 0) (at 151.765 165.1 0)
+      (effects (font (size 1.27 1.27)) hide)
+    )
+    (property "Value" "GND" (id 1) (at 151.765 162.56 0))
+    (property "Footprint" "" (id 2) (at 151.765 158.75 0)
+      (effects (font (size 1.27 1.27)) hide)
+    )
+    (property "Datasheet" "" (id 3) (at 151.765 158.75 0)
+      (effects (font (size 1.27 1.27)) hide)
+    )
+    (pin "1")
+  )
   (symbol (lib_id "power:PWR_FLAG") (at 168.275 205.105 0) (unit 1)
     (in_bom yes) (on_board yes)
@@
     (pin "2")
   )
+  (symbol (lib_id "Device:LED_Small_Filled") (at 151.765 155.575 90) (unit 1)
+    (in_bom yes) (on_board yes)
+    (property "Reference" "D25" (id 0) (at 146.685 154.94 90)
+      (effects (font (size 1.27 1.27)) (justify right))
+    )
+    (property "Value" "OUT 1" (id 1) (at 144.145 156.845 90)
+      (effects (font (size 1.27 1.27)) (justify right))
+    )
+    (property "Footprint" "LED_SMD:LED_0603_1608Metric" (id 2) (at 151.765 155.575 90)
+      (effects (font (size 1.27 1.27)) hide)
+    )
+    (property "Datasheet" "~" (id 3) (at 151.765 155.575 90)
+      (effects (font (size 1.27 1.27)) hide)
+    )
+    (pin "1")
+    (pin "2")
+  )
   (symbol (lib_id "Device:R_Small") (at 100.33 186.055 0) (mirror y) (unit 1)
     (in_bom yes) (on_board yes)
@@
       (reference "#PWR021") (unit 1) (value "GND") (footprint "")
     )
+    (path "/b0286384-6b2d-48c1-9cf1-743ec9ceba55"
+      (reference "#PWR022") (unit 1) (value "GND") (footprint "")
+    )
     (path "/00000000-0000-0000-0000-000062d02e9a"
       (reference "#PWR023") (unit 1) (value "+12V") (footprint "")
@@
       (reference "D24") (unit 1) (value "PMEG3050EP") (footprint "Diode_SMD:D_SOD-128")
     )
+    (path "/dfd17e1c-447d-41fd-bb31-23d497ec113b"
+      (reference "D25") (unit 1) (value "OUT 1") (footprint "LED_SMD:LED_0603_1608Metric")
+    )
     (path "/fbb50421-f88c-4d82-969c-09c2a9fef6a9"
       (reference "F1") (unit 1) (value "Fuse_Small") (footprint "Resistor_SMD:R_0805_2012Metric_Pad1.20x1.40mm_HandSolder")
@@
       (reference "R55") (unit 1) (value "140m") (footprint "Resistor_SMD:R_0805_2012Metric")
     )
+    (path "/ae0697cf-c6d2-46a1-8e04-37ae584a03eb"
+      (reference "R56") (unit 1) (value "120") (footprint "Resistor_SMD:R_0603_1608Metric")
+    )
     (path "/00000000-0000-0000-0000-000061b3409a"
