File: uHoubolt_PCB_PMU.kicad_sch (KiCad schematic)
At the start: 118 parts, among them J10 Debug, J11 AltimaxPwr, J12 CAN1, J13 CAN2, J14 CAN1, J15 CAN2, J16 CAN1, J17 CAN2, J18 CAN1, J19 CAN2, J2 Battery, J23 Payload, J25 RCU, J27 Umbilical0, J28 Umbilical0, J29 AltimaxArm, J3 Power, J4 BatteryAltimax, J5 Umbilical1, J6 AltimaxArm, J8 Altimax_PWR, J9 Debug, Q1 BSZ0905PNSATMA1, Q2 BSZ0902NSATMA1, Q3 SISA88DN or similar, SW1 Power_1, SW2 Power_2, SW3 Pyro_1, SW4 Pyro_2, U1 LM5069, U10 ICM-20602, U11 LPS25HB, U12 SFH617A-1X007T, U14 LiIon_Charger, U15 SFH617A-1X007T, U2 LMP8640 F, U4 LiIon_Charger, U5 STM32G491MET6-LQFP80, U6 W25Q256JV, U7 MCP1700-3302E, U8 MCP2562FDx-x_MF, U9 MCP2562FDx-x_MF, X1 TXC-7C

Commit message: V3 Updated ready for check
Parts:
- removed J11: AltimaxPwr, TXV_Library_Footprints:Molex_SL_1x2_Vertical, symbol Connector_Generic:Conn_01x02
- removed J29: AltimaxArm, TXV_Library_Footprints:Molex_Nano-Fit_105309-xx02_1x02_P2.50mm_Vertical, symbol Connector_Generic:Conn_01x02
- removed J6: AltimaxArm, TXV_Library_Footprints:Molex_SL_1x2_Vertical, symbol Connector_Generic:Conn_01x02
- removed J8: Altimax_PWR, TXV_Library_Footprints:Molex_SL_1x2_Vertical, symbol Connector_Generic:Conn_01x02
- added J1, J7: Conn_01x04, TXV_Library_Footprints:Molex_Nano-Fit_105309-xx04_1x04_P2.50mm_Vertical, symbol Connector_Generic:Conn_01x04
Connections:
- net +12V: now also J7.1 (Pin_1)
- net GND: now also J7.2 (Pin_2)
- net GND_Altimax: now also J1.2 (Pin_2)
- net at SW2.2 (B): now also J1.1 (Pin_1)
- net at SW4.1 (A): now also J1.4 (Pin_4)
- net at SW4.2 (B): now also J1.3 (Pin_3)
- net at U15.4: now also J7.3 (Pin_3)
- net at U15.3: now also J7.4 (Pin_4)
Other:
- moved on the sheet: SW4

Commit message: V3 2. Update ready for check
Changed lines of the file:
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@@
+    (stroke (width 0) (type default) (color 0 0 0 0))
+  )
+  (wire (pts (xy 117.475 132.08) (xy 118.11 132.08))
     (stroke (width 0) (type default) (color 0 0 0 0))
   )
@@
     (stroke (width 0) (type default) (color 0 0 0 0))
   )
-  (wire (pts (xy 118.11 118.11) (xy 118.11 132.08))
+  (wire (pts (xy 117.475 118.11) (xy 117.475 132.08))
     (stroke (width 0) (type default) (color 0 0 0 0))
   )
@@
     (stroke (width 0) (type default) (color 0 0 0 0))
   )
-  (wire (pts (xy 116.84 118.11) (xy 118.11 118.11))
-    (stroke (width 0) (type default) (color 0 0 0 0))
-  )
+  (wire (pts (xy 116.84 118.11) (xy 117.475 118.11))
+    (stroke (width 0) (type default) (color 0 0 0 0))
+  )
