File: Output.kicad_sch (KiCad schematic)
At the start: 8 parts, among them J20 Output, Q4 SISA88DN or similar

Commit message: V3 2. Update ready for check
Parts:
- renumbered D10 to D12, D11 to D13, J20 to J21, JP4 to JP5, Q4 to Q5, R32 to R35, R33 to R36, R34 to R37
Changed lines of the file:
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@@
   (symbol (lib_id "Jumper:Jumper_3_Open") (at 151.765 62.23 0)
     (in_bom yes) (on_board yes) (fields_autoplaced)
-    (property "Reference" "JP4" (id 0) (at 151.765 58.42 0))
+    (property "Reference" "JP5" (id 0) (at 151.765 58.42 0))
     (property "Value" "Jumper_3_Open" (id 1) (at 151.765 58.42 0)
       (effects (font (size 1.27 1.27)) hide)
@@
   (symbol (lib_id "Device:Q_NMOS_GDS") (at 149.225 78.74 0)
     (in_bom yes) (on_board yes)
-    (property "Reference" "Q4" (id 0) (at 154.432 77.5716 0)
+    (property "Reference" "Q5" (id 0) (at 154.432 77.5716 0)
       (effects (font (size 1.27 1.27)) (justify left))
     )
@@
   (symbol (lib_id "Device:D_Schottky_Small_Filled") (at 149.225 69.85 90) (mirror x)
     (in_bom yes) (on_board yes)
-    (property "Reference" "D11" (id 0) (at 144.145 68.58 90)
+    (property "Reference" "D13" (id 0) (at 144.145 68.58 90)
       (effects (font (size 1.27 1.27)) (justify right))
     )
@@
   (symbol (lib_id "Device:R_Small") (at 133.35 81.915 0)
     (in_bom yes) (on_board yes)
-    (property "Reference" "R32" (id 0) (at 130.175 81.28 0))
+    (property "Reference" "R35" (id 0) (at 130.175 81.28 0))
     (property "Value" "120" (id 1) (at 130.175 83.185 0))
     (property "Footprint" "Resistor_SMD:R_0603_1608Metric" (id 2) (at 133.35 81.915 0)
@@
   (symbol (lib_id "Connector_Generic:Conn_01x02") (at 157.48 68.58 0)
     (in_bom yes) (on_board yes)
-    (property "Reference" "J20" (id 0) (at 159.512 68.7832 0)
+    (property "Reference" "J21" (id 0) (at 159.512 68.7832 0)
       (effects (font (size 1.27 1.27)) (justify left))
     )
@@
   (symbol (lib_id "Device:R_Small") (at 137.16 81.915 180)
     (in_bom yes) (on_board yes)
-    (property "Reference" "R33" (id 0) (at 138.43 81.28 0)
+    (property "Reference" "R36" (id 0) (at 138.43 81.28 0)
       (effects (font (size 1.27 1.27)) (justify right))
     )
@@
   (symbol (lib_id "Device:LED_Small_Filled") (at 133.35 87.63 90)
     (in_bom yes) (on_board yes)
-    (property "Reference" "D10" (id 0) (at 128.27 86.995 90)
+    (property "Reference" "D12" (id 0) (at 128.27 86.995 90)
       (effects (font (size 1.27 1.27)) (justify right))
     )
@@
   (symbol (lib_id "Device:R_Small") (at 140.97 78.74 90)
     (in_bom yes) (on_board yes)
-    (property "Reference" "R34" (id 0) (at 140.97 74.93 90))
+    (property "Reference" "R37" (id 0) (at 140.97 74.93 90))
     (property "Value" "120" (id 1) (at 140.97 76.835 90))
     (property "Footprint" "Resistor_SMD:R_0603_1608Metric" (id 2) (at 140.97 78.74 0)

Commit message: Update of v3
Changed the silkscreen + more pads
Parts:
- renumbered D12 to D17, D13 to D18, J21 to J24, JP5 to JP7, Q5 to Q7, R35 to R42, R36 to R48, R37 to R49
Changed lines of the file:
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@@
   (symbol (lib_id "Jumper:Jumper_3_Open") (at 151.765 62.23 0)
     (in_bom yes) (on_board yes) (fields_autoplaced)
-    (property "Reference" "JP5" (id 0) (at 151.765 58.42 0))
+    (property "Reference" "JP7" (id 0) (at 151.765 58.42 0))
     (property "Value" "Jumper_3_Open" (id 1) (at 151.765 58.42 0)
       (effects (font (size 1.27 1.27)) hide)
@@
   (symbol (lib_id "Device:Q_NMOS_GDS") (at 149.225 78.74 0)
     (in_bom yes) (on_board yes)
-    (property "Reference" "Q5" (id 0) (at 154.432 77.5716 0)
+    (property "Reference" "Q7" (id 0) (at 154.432 77.5716 0)
       (effects (font (size 1.27 1.27)) (justify left))
     )
@@
   (symbol (lib_id "Device:D_Schottky_Small_Filled") (at 149.225 69.85 90) (mirror x)
     (in_bom yes) (on_board yes)
-    (property "Reference" "D13" (id 0) (at 144.145 68.58 90)
+    (property "Reference" "D18" (id 0) (at 144.145 68.58 90)
       (effects (font (size 1.27 1.27)) (justify right))
     )
@@
   (symbol (lib_id "Device:R_Small") (at 133.35 81.915 0)
     (in_bom yes) (on_board yes)
-    (property "Reference" "R35" (id 0) (at 130.175 81.28 0))
+    (property "Reference" "R42" (id 0) (at 130.175 81.28 0))
     (property "Value" "120" (id 1) (at 130.175 83.185 0))
     (property "Footprint" "Resistor_SMD:R_0603_1608Metric" (id 2) (at 133.35 81.915 0)
@@
   (symbol (lib_id "Connector_Generic:Conn_01x02") (at 157.48 68.58 0)
     (in_bom yes) (on_board yes)
-    (property "Reference" "J21" (id 0) (at 159.512 68.7832 0)
+    (property "Reference" "J24" (id 0) (at 159.512 68.7832 0)
       (effects (font (size 1.27 1.27)) (justify left))
     )
@@
   (symbol (lib_id "Device:R_Small") (at 137.16 81.915 180)
     (in_bom yes) (on_board yes)
-    (property "Reference" "R36" (id 0) (at 138.43 81.28 0)
+    (property "Reference" "R48" (id 0) (at 138.43 81.28 0)
       (effects (font (size 1.27 1.27)) (justify right))
     )
@@
   (symbol (lib_id "Device:LED_Small_Filled") (at 133.35 87.63 90)
     (in_bom yes) (on_board yes)
-    (property "Reference" "D12" (id 0) (at 128.27 86.995 90)
+    (property "Reference" "D17" (id 0) (at 128.27 86.995 90)
       (effects (font (size 1.27 1.27)) (justify right))
     )
@@
   (symbol (lib_id "Device:R_Small") (at 140.97 78.74 90)
     (in_bom yes) (on_board yes)
-    (property "Reference" "R37" (id 0) (at 140.97 74.93 90))
+    (property "Reference" "R49" (id 0) (at 140.97 74.93 90))
     (property "Value" "120" (id 1) (at 140.97 76.835 90))
     (property "Footprint" "Resistor_SMD:R_0603_1608Metric" (id 2) (at 140.97 78.74 0)
